Commit message: camera_color_frameとcamera_color_optical_frameを追加

File: crane_plus_description/urdf/camera.urdf.xacro (robot description, xacro)
@@ -2,4 +2,5 @@
 <robot name="camera" xmlns:xacro="http://www.ros.org/wiki/xacro">
   <xacro:macro name="sensor_camera" params="parent">
+    <xacro:property name="M_PI" value="3.1415926535897931" />
     <link name="camera_link">
       <visual>
@@ -16,4 +17,16 @@
       <child link="camera_link" />
     </joint>
+    <link name="camera_color_frame" />
+    <joint name="camera_color_joint" type="fixed">
+      <origin xyz="0 0 0" rpy="0 0 0" />
+      <parent link="camera_link" />
+      <child link="camera_color_frame" />
+    </joint>
+    <link name="camera_color_optical_frame" />
+    <joint name="camera_color_optical_joint" type="fixed">
+      <origin xyz="0 0 0" rpy="0 ${M_PI} ${M_PI/2}" />
+      <parent link="camera_color_frame" />
+      <child link="camera_color_optical_frame" />
+    </joint>
   </xacro:macro>
 </robot>

Commit message: M_PIからradiansに変更

File: crane_plus_description/urdf/camera.urdf.xacro (robot description, xacro)
@@ -2,5 +2,4 @@
 <robot name="camera" xmlns:xacro="http://www.ros.org/wiki/xacro">
   <xacro:macro name="sensor_camera" params="parent">
-    <xacro:property name="M_PI" value="3.1415926535897931" />
     <link name="camera_link">
       <visual>
@@ -25,5 +24,5 @@
     <link name="camera_color_optical_frame" />
     <joint name="camera_color_optical_joint" type="fixed">
-      <origin xyz="0 0 0" rpy="0 ${M_PI} ${M_PI/2}" />
+	    <origin xyz="0 0 0" rpy="0 ${radians(180)} ${radians(90)}" />
       <parent link="camera_color_frame" />
       <child link="camera_color_optical_frame" />

Commit message: tabをspaceに置換、インデントを修正

File: crane_plus_description/urdf/camera.urdf.xacro (robot description, xacro)
@@ -8,5 +8,5 @@
           <box size="0.05 0.05 0.05" />
         </geometry>
-	<material name="Black" />
+  <material name="Black" />
       </visual>
     </link>
@@ -24,5 +24,5 @@
     <link name="camera_color_optical_frame" />
     <joint name="camera_color_optical_joint" type="fixed">
-	    <origin xyz="0 0 0" rpy="0 ${radians(180)} ${radians(90)}" />
+      <origin xyz="0 0 0" rpy="0 ${radians(180)} ${radians(90)}" />
       <parent link="camera_color_frame" />
       <child link="camera_color_optical_frame" />

File: crane_plus_description/urdf/camera_stand.urdf.xacro (robot description, xacro)
@@ -8,6 +8,6 @@
           <box size="0.02 0.02 0.285" />
         </geometry>
-	<material name="grey">
-	  <color rgba="0.8 0.8 0.8 1.0" />
+        <material name="grey">
+          <color rgba="0.8 0.8 0.8 1.0" />
         </material>
       </visual>
@@ -24,6 +24,6 @@
           <box size="0.02 0.02 0.44" />
         </geometry>
-	<material name="grey">
-	  <color rgba="0.8 0.8 0.8 1.0" />
+        <material name="grey">
+          <color rgba="0.8 0.8 0.8 1.0" />
         </material>
       </visual>
@@ -40,6 +40,6 @@
           <box size="0.02 0.02 0.13" />
         </geometry>
-	<material name="grey">
-	  <color rgba="0.8 0.8 0.8 1.0" />
+        <material name="grey">
+          <color rgba="0.8 0.8 0.8 1.0" />
         </material>
       </visual>
@@ -56,6 +56,6 @@
           <box size="0.02 0.02 0.13" />
         </geometry>
-	<material name="grey">
-	  <color rgba="0.8 0.8 0.8 1.0" />
+        <material name="grey">
+          <color rgba="0.8 0.8 0.8 1.0" />
         </material>
       </visual>
@@ -72,6 +72,6 @@
           <box size="0.02 0.02 0.13" />
         </geometry>
-	<material name="grey">
-	  <color rgba="0.8 0.8 0.8 1.0" />
+        <material name="grey">
+          <color rgba="0.8 0.8 0.8 1.0" />
         </material>
       </visual>
@@ -88,6 +88,6 @@
           <box size="0.02 0.02 0.13" />
         </geometry>
-	<material name="grey">
-	  <color rgba="0.8 0.8 0.8 1.0" />
+        <material name="grey">
+          <color rgba="0.8 0.8 0.8 1.0" />
         </material>
       </visual>

File: crane_plus_description/urdf/crane_plus.xacro (robot description, xacro)
@@ -58,5 +58,5 @@
               joint_hand_lower_limit
               joint_hand_upper_limit
-	      use_camera
+              use_camera
               *origin">
     <joint name="${name_joint_base}" type="fixed">

Commit message: インデントを修正

File: crane_plus_description/urdf/camera.urdf.xacro (robot description, xacro)
@@ -8,5 +8,5 @@
           <box size="0.05 0.05 0.05" />
         </geometry>
-  <material name="Black" />
+        <material name="Black" />
       </visual>
     </link>

Commit message: 新しいカメラスタンドに対応

File: crane_plus_description/urdf/camera.urdf.xacro (robot description, xacro)
@@ -12,5 +12,5 @@
     </link>
     <joint name="camera_joint" type="fixed">
-      <origin xyz="0.1030 0.1025 0.4600" rpy="0 0 0" />
+      <origin xyz="0.103 0.1025 0.48" rpy="0 0 0" />
       <parent link="${parent}" />
       <child link="camera_link" />

File: crane_plus_description/urdf/camera_stand.urdf.xacro (robot description, xacro)
@@ -14,5 +14,5 @@
     </link>
     <joint name="camera_stand_joint1" type="fixed">
-      <origin xyz="-0.05 0.08 0" rpy="${radians(90)} 0 0" />
+      <origin xyz="-0.05 0.08 0.01" rpy="${radians(90)} 0 0" />
       <parent link="${parent}" />
       <child link="camera_stand_p1" />
@@ -30,5 +30,5 @@
     </link>
     <joint name="camera_stand_joint2" type="fixed">
-      <origin xyz="-0.05 0.1025 0.23" rpy="0 0 0" />
+      <origin xyz="-0.05 0.1025 0.24" rpy="0 0 0" />
       <parent link="${parent}" />
       <child link="camera_stand_p2" />
@@ -46,5 +46,5 @@
     </link>
     <joint name="camera_stand_joint3" type="fixed">
-      <origin xyz="0.02 0.1025 0.44" rpy="0 ${radians(90)} 0" />
+      <origin xyz="0.02 0.1025 0.45" rpy="0 ${radians(90)} 0" />
       <parent link="${parent}" />
       <child link="camera_stand_p3" />
@@ -54,5 +54,5 @@
         <origin xyz="0 0 0" rpy="0 0 0" />
         <geometry>
-          <box size="0.02 0.02 0.13" />
+          <box size="0.02 0.02 0.05" />
         </geometry>
         <material name="grey">
@@ -62,5 +62,5 @@
     </link>
     <joint name="camera_stand_joint4" type="fixed">
-      <origin xyz="0.02 -0.0525 0" rpy="0 ${radians(90)} 0" />
+      <origin xyz="-0.015 -0.0525 0.01" rpy="0 ${radians(90)} 0" />
       <parent link="${parent}" />
       <child link="camera_stand_p4" />
@@ -70,5 +70,5 @@
         <origin xyz="0 0 0" rpy="0 0 0" />
         <geometry>
-          <box size="0.02 0.02 0.13" />
+          <box size="0.02 0.02 0.05" />
         </geometry>
         <material name="grey">
@@ -78,24 +78,8 @@
     </link>
     <joint name="camera_stand_joint5" type="fixed">
-      <origin xyz="0.02 0.0525 0" rpy="0 ${radians(90)} 0" />
+      <origin xyz="-0.015 0.2125 0.01" rpy="0 ${radians(90)} 0" />
       <parent link="${parent}" />
       <child link="camera_stand_p5" />
     </joint>
-    <link name="camera_stand_p6">
-      <visual>
-        <origin xyz="0 0 0" rpy="0 0 0" />
-        <geometry>
-          <box size="0.02 0.02 0.13" />
-        </geometry>
-        <material name="grey">
-          <color rgba="0.8 0.8 0.8 1.0" />
-        </material>
-      </visual>
-    </link>
-    <joint name="camera_stand_joint6" type="fixed">
-      <origin xyz="0.02 0.2125 0" rpy="0 ${radians(90)} 0" />
-      <parent link="${parent}" />
-      <child link="camera_stand_p6" />
-    </joint>
   </xacro:macro>
 </robot>

Commit message: Update crane_plus_description/urdf/camera.urdf.xacro
Co-authored-by: Kuwamai <kuwagata@rt-net.jp>

File: crane_plus_description/urdf/camera.urdf.xacro (robot description, xacro)
@@ -12,5 +12,5 @@
     </link>
     <joint name="camera_joint" type="fixed">
-      <origin xyz="0.103 0.1025 0.48" rpy="0 0 0" />
+      <origin xyz="0.103 0.1025 0.46" rpy="0 0 0" />
       <parent link="${parent}" />
       <child link="camera_link" />

Commit message: 色検出サンプルの追加 (#54)
* 色認識して位置をtfに送信

* ピックアンドプレイスの実装

* colcon testで確認修正済み

* カメラのキャリブレーション結果を用いて把持対象物の位置を算出

* 変数名をsnake_caseに統一

* image_geometryを追加

* 100文字を超える行の折返し

* highgui関連の行を削除

* コメントの追記と変更

* 画像処理のコードを整理

* コメントを修正

* frame_idの名前をtarget_0に変更

* launchファイルで色認識とピックアンドプレースを実行

* カメラサンプル用のlaunchファイルを作成

* 二行空け

* 三行空け

* 二行空けでcolcon testをパス

* control_gripper関数のコメントを追加

Co-authored-by: Kuwamai <kuwagata@rt-net.jp>

* control_arm関数のコメントを追加

Co-authored-by: Kuwamai <kuwagata@rt-net.jp>

* tf取得処理のコメントを修正

Co-authored-by: Kuwamai <kuwagata@rt-net.jp>

* camera_info.yamlをconfigディレクトリに配置してlaunch実行時に読み込む

* コメントを修正

* HSVのHの最大値を179に設定

* カメラサンプルの説明を追加

* 赤色を認識するためにマスク画像を2つ生成して合成

* HSVの値を調整

* 不正確なコメントを修正

Co-authored-by: Kuwamai <kuwagata@rt-net.jp>

* 閾値の画像を配信

* RViz起動時に二値化画像を表示

* colcon testをパス

* キャリブレーションを行って作成したカメラのパラメータファイルを追加

* 新しいカメラスタンドに対応

* 色検出サンプルを修正

* 認識を検出に変更

* ARマーカ検出サンプルを移植

* Revert "ARマーカ検出サンプルを移植"

This reverts commit 0a15ed7a4a7da803c47f3296be58cc408d80885c.

* Update crane_plus_description/urdf/camera.urdf.xacro

Co-authored-by: Kuwamai <kuwagata@rt-net.jp>

* Update crane_plus_examples/src/color_detection.cpp

Co-authored-by: Kuwamai <kuwagata@rt-net.jp>

* Update crane_plus_examples/src/color_detection.cpp

Co-authored-by: Kuwamai <kuwagata@rt-net.jp>

* Update crane_plus_examples/src/pick_and_place_tf.cpp

Co-authored-by: Kuwamai <kuwagata@rt-net.jp>

* Update crane_plus_examples/src/pick_and_place_tf.cpp

Co-authored-by: Kuwamai <kuwagata@rt-net.jp>

* レビューコメントに対応

* 手先を水平にして把持を行う

* 余分なTABを削除

* 余分なコメントを削除

* 待機姿勢を手先だけ真上に向けるように変更（拘束条件も追加）

* 「掴む準備をする」姿勢を削除

* 把持した物体をカメラの画角外に置くように変更

* コメントアウトしていた「掴む準備をする」姿勢を削除

* RViz上のviewsを削除

---------

Co-authored-by: Kuwamai <kuwagata@rt-net.jp>

File: crane_plus_description/urdf/camera.urdf.xacro (robot description, xacro)
@@ -12,5 +12,5 @@
     </link>
     <joint name="camera_joint" type="fixed">
-      <origin xyz="0.1030 0.1025 0.4600" rpy="0 0 0" />
+      <origin xyz="0.103 0.1025 0.46" rpy="0 0 0" />
       <parent link="${parent}" />
       <child link="camera_link" />

Commit message: カメラ追加

File: crane_plus_description/urdf/camera.urdf.xacro (robot description, xacro)
@@ -8,5 +8,7 @@
           <box size="0.05 0.05 0.05" />
         </geometry>
-        <material name="Black" />
+        <material name="black">
+          <color rgba="0.2 0.2 0.2 1.0"/>
+        </material>
       </visual>
     </link>

File: crane_plus_description/urdf/camera_stand.urdf.xacro (robot description, xacro)
@@ -12,4 +12,10 @@
         </material>
       </visual>
+      <collision>
+        <origin xyz="0 0 0" rpy="0 0 0"/>
+        <geometry>
+          <box size="0.02 0.02 0.285" />
+        </geometry>
+      </collision>
     </link>
     <joint name="camera_stand_joint1" type="fixed">
@@ -28,4 +34,10 @@
         </material>
       </visual>
+      <collision>
+        <origin xyz="0 0 0" rpy="0 0 0"/>
+        <geometry>
+          <box size="0.02 0.02 0.44" />
+        </geometry>
+      </collision>
     </link>
     <joint name="camera_stand_joint2" type="fixed">
@@ -44,4 +56,10 @@
         </material>
       </visual>
+      <collision>
+        <origin xyz="0 0 0" rpy="0 0 0"/>
+        <geometry>
+          <box size="0.02 0.02 0.13" />
+        </geometry>
+      </collision>
     </link>
     <joint name="camera_stand_joint3" type="fixed">
@@ -60,4 +78,10 @@
         </material>
       </visual>
+      <collision>
+        <origin xyz="0 0 0" rpy="0 0 0"/>
+        <geometry>
+          <box size="0.02 0.02 0.05" />
+        </geometry>
+      </collision>
     </link>
     <joint name="camera_stand_joint4" type="fixed">
@@ -76,4 +100,10 @@
         </material>
       </visual>
+      <collision>
+        <origin xyz="0 0 0" rpy="0 0 0"/>
+        <geometry>
+          <box size="0.02 0.02 0.05" />
+        </geometry>
+      </collision>
     </link>
     <joint name="camera_stand_joint5" type="fixed">

File: crane_plus_description/urdf/crane_plus.gazebo.xacro (robot description, xacro)
@@ -24,4 +24,5 @@
             name_link_4
             name_link_hand
+            use_camera
             use_ignition
             config_package
@@ -71,4 +72,52 @@
       <xacro:material_gazebo_white/>
     </gazebo>
+    <xacro:if value="$(arg use_camera)">
+      <gazebo>
+        <plugin filename="ignition-gazebo-sensors-system" name="ignition::gazebo::systems::Sensors">
+          <render_engine>ogre2</render_engine>
+        </plugin>
+      </gazebo>
+      <gazebo reference="camera_color_optical_frame">
+        <sensor name="camera" type="camera">
+          <pose relative_to="camera_color_optical_frame">0 0 0 ${radians(90)} ${radians(-90)} 0</pose>
+          <update_rate>10</update_rate>
+          <always_on>true</always_on>
+          <topic>image_raw</topic>
+          <gz_frame_id>camera_color_optical_frame</gz_frame_id>
+          <camera name="camera">
+            <xacro:property name="camera_width" value="640"/>
+            <xacro:property name="camera_height" value="480"/>
+            <xacro:property name="camera_hfov" value="${radians(120)}"/>
+            <xacro:property name="camera_focal_length" value="${camera_width / (2 * tan(camera_hfov / 2))}"/>
+            <horizontal_fov>${camera_hfov}</horizontal_fov>
+            <image>
+              <width>${camera_width}</width>
+              <height>${camera_height}</height>
+            </image>
+            <clip>
+              <near>0.1</near>
+              <far>10.0</far>
+            </clip>
+            <lens>
+              <intrinsics>
+                <fx>${camera_focal_length}</fx>
+                <fy>${camera_focal_length}</fy>
+                <cx>${(camera_width + 1) / 2}</cx>
+                <cy>${(camera_height + 1) / 2}</cy>
+                <s>1.0</s>
+              </intrinsics>
+              <projection>
+                <p_fx>${camera_focal_length}</p_fx>
+                <p_fy>${camera_focal_length}</p_fy>
+                <p_cx>${(camera_width + 1) / 2}</p_cx>
+                <p_cy>${(camera_height + 1) / 2}</p_cy>
+                <tx>0</tx>
+                <ty>0</ty>
+              </projection>
+            </lens>
+          </camera>
+        </sensor>
+      </gazebo>
+    </xacro:if>
   </xacro:macro>
 </robot>

File: crane_plus_description/urdf/crane_plus.urdf.xacro (robot description, xacro)
@@ -118,4 +118,5 @@
       name_link_4="${NAME_LINK_4}"
       name_link_hand="${NAME_LINK_HAND}"
+      use_camera="$(arg use_camera)"
       use_ignition="$(arg use_ignition)"
       config_package="$(arg gz_control_config_package)"

Commit message: カメラスタンドのURDF修正

File: crane_plus_description/urdf/camera.urdf.xacro (robot description, xacro)
@@ -6,5 +6,5 @@
         <origin xyz="0 0 0" rpy="0 0 0" />
         <geometry>
-          <box size="0.05 0.05 0.05" />
+          <box size="0.03 0.08 0.05" />
         </geometry>
         <material name="black">
@@ -12,7 +12,13 @@
         </material>
       </visual>
+      <collision>
+        <origin xyz="0 0 0" rpy="0 0 0"/>
+        <geometry>
+          <box size="0.03 0.08 0.05" />
+        </geometry>
+      </collision>
     </link>
     <joint name="camera_joint" type="fixed">
-      <origin xyz="0.103 0.1025 0.46" rpy="0 0 0" />
+      <origin xyz="0.10626 0.10253 0.46" rpy="0 0 0" />
       <parent link="${parent}" />
       <child link="camera_link" />

File: crane_plus_description/urdf/camera_stand.urdf.xacro (robot description, xacro)
@@ -6,5 +6,5 @@
         <origin xyz="0 0 0" rpy="0 0 0" />
         <geometry>
-          <box size="0.02 0.02 0.285" />
+          <box size="0.02 0.285 0.02" />
         </geometry>
         <material name="grey">
@@ -15,10 +15,10 @@
         <origin xyz="0 0 0" rpy="0 0 0"/>
         <geometry>
-          <box size="0.02 0.02 0.285" />
+          <box size="0.02 0.285 0.02" />
         </geometry>
       </collision>
     </link>
     <joint name="camera_stand_joint1" type="fixed">
-      <origin xyz="-0.05 0.08 0.01" rpy="${radians(90)} 0 0" />
+      <origin xyz="-0.052 0.08 0.01" rpy="0 0 0" />
       <parent link="${parent}" />
       <child link="camera_stand_p1" />
@@ -42,6 +42,6 @@
     </link>
     <joint name="camera_stand_joint2" type="fixed">
-      <origin xyz="-0.05 0.1025 0.24" rpy="0 0 0" />
-      <parent link="${parent}" />
+      <origin xyz="0 0.02253 0.23" rpy="0 0 0" />
+      <parent link="camera_stand_p1" />
       <child link="camera_stand_p2" />
     </joint>
@@ -50,5 +50,5 @@
         <origin xyz="0 0 0" rpy="0 0 0" />
         <geometry>
-          <box size="0.02 0.02 0.13" />
+          <box size="0.13 0.02 0.02" />
         </geometry>
         <material name="grey">
@@ -59,11 +59,11 @@
         <origin xyz="0 0 0" rpy="0 0 0"/>
         <geometry>
-          <box size="0.02 0.02 0.13" />
+          <box size="0.129 0.02 0.02" />
         </geometry>
       </collision>
     </link>
     <joint name="camera_stand_joint3" type="fixed">
-      <origin xyz="0.02 0.1025 0.45" rpy="0 ${radians(90)} 0" />
-      <parent link="${parent}" />
+      <origin xyz="0.075 0 0.21" rpy="0 0 0" />
+      <parent link="camera_stand_p2" />
       <child link="camera_stand_p3" />
     </joint>
@@ -72,5 +72,5 @@
         <origin xyz="0 0 0" rpy="0 0 0" />
         <geometry>
-          <box size="0.02 0.02 0.05" />
+          <box size="0.055 0.02 0.02" />
         </geometry>
         <material name="grey">
@@ -81,11 +81,11 @@
         <origin xyz="0 0 0" rpy="0 0 0"/>
         <geometry>
-          <box size="0.02 0.02 0.05" />
+          <box size="0.054 0.019 0.02" />
         </geometry>
       </collision>
     </link>
     <joint name="camera_stand_joint4" type="fixed">
-      <origin xyz="-0.015 -0.0525 0.01" rpy="0 ${radians(90)} 0" />
-      <parent link="${parent}" />
+      <origin xyz="0.0375 -0.1325 0" rpy="0 0 0" />
+      <parent link="camera_stand_p1" />
       <child link="camera_stand_p4" />
     </joint>
@@ -94,5 +94,5 @@
         <origin xyz="0 0 0" rpy="0 0 0" />
         <geometry>
-          <box size="0.02 0.02 0.05" />
+          <box size="0.055 0.02 0.02" />
         </geometry>
         <material name="grey">
@@ -103,11 +103,11 @@
         <origin xyz="0 0 0" rpy="0 0 0"/>
         <geometry>
-          <box size="0.02 0.02 0.05" />
+          <box size="0.054 0.02 0.02" />
         </geometry>
       </collision>
     </link>
     <joint name="camera_stand_joint5" type="fixed">
-      <origin xyz="-0.015 0.2125 0.01" rpy="0 ${radians(90)} 0" />
-      <parent link="${parent}" />
+      <origin xyz="0.0375 0.1325 0" rpy="0 0 0" />
+      <parent link="camera_stand_p1" />
       <child link="camera_stand_p5" />
     </joint>
