Commit message: Remove gripper model parameters

File: crane_plus_description/urdf/crane_plus.gazebo.xacro (robot description, xacro)
@@ -35,20 +35,12 @@
     </gazebo>
     <gazebo reference="${name_link_4}">
-      <!-- <mu1>10.0</mu1>
-      <mu2>100.0</mu2> -->
-      <min_depth>0.001</min_depth>
-      <maxVel>0</maxVel>
-      <kp>100000</kp>
-      <kd>100</kd>
-      <material>Gazebo/Green</material>
+      <mu1>0.2</mu1>
+      <mu2>0.2</mu2>
+      <material>Gazebo/Black</material>
     </gazebo>
     <gazebo reference="${name_link_hand}">
-      <!-- <mu1>10.0</mu1>
-      <mu2>100.0</mu2> -->
-      <min_depth>0.001</min_depth>
-      <maxVel>0</maxVel>
-      <kp>100000</kp>
-      <kd>100</kd>
-      <material>Gazebo/Green</material>
+      <mu1>0.2</mu1>
+      <mu2>0.2</mu2>
+      <material>Gazebo/White</material>
     </gazebo>
   </xacro:macro>

Commit message: gazebo.materialスクリプトが読み込まれないため、パラメータを変更

File: crane_plus_description/urdf/crane_plus.gazebo.xacro (robot description, xacro)
@@ -1,4 +1,22 @@
 <?xml version="1.0"?>
 <robot xmlns:xacro="http://www.ros.org/wiki/xacro">
+  <xacro:macro name="material_gazebo_black">
+    <visual>
+      <material>
+        <ambient>0 0 0 1</ambient>
+        <diffuse>0 0 0 1</diffuse>
+        <specular>0.1 0.1 0.1 5.0</specular>
+      </material>
+    </visual>
+  </xacro:macro>
+  <xacro:macro name="material_gazebo_white">
+    <visual>
+      <material>
+        <ambient>1 1 1 1</ambient>
+        <diffuse>1 1 1 1</diffuse>
+        <specular>0.1 0.1 0.1 128.0</specular>
+      </material>
+    </visual>
+  </xacro:macro>
   <xacro:macro name="gazebo_robot_settings"
     params="name_link_base
@@ -19,30 +37,30 @@
       <mu1>0.2</mu1>
       <mu2>0.2</mu2>
-      <material>Gazebo/Black</material>
+      <xacro:material_gazebo_black/>
     </gazebo>
     <gazebo reference="${name_link_1}">
       <mu1>0.2</mu1>
       <mu2>0.2</mu2>
-      <material>Gazebo/White</material>
+      <xacro:material_gazebo_white/>
     </gazebo>
     <gazebo reference="${name_link_2}">
       <mu1>0.2</mu1>
       <mu2>0.2</mu2>
-      <material>Gazebo/Black</material>
+      <xacro:material_gazebo_black/>
     </gazebo>
     <gazebo reference="${name_link_3}">
       <mu1>0.2</mu1>
       <mu2>0.2</mu2>
-      <material>Gazebo/White</material>
+      <xacro:material_gazebo_white/>
     </gazebo>
     <gazebo reference="${name_link_4}">
       <mu1>0.2</mu1>
       <mu2>0.2</mu2>
-      <material>Gazebo/Black</material>
+      <xacro:material_gazebo_black/>
     </gazebo>
     <gazebo reference="${name_link_hand}">
       <mu1>0.2</mu1>
       <mu2>0.2</mu2>
-      <material>Gazebo/White</material>
+      <xacro:material_gazebo_white/>
     </gazebo>
   </xacro:macro>

Commit message: crane_plus_ignition パッケージを追加し、Gazeboの使用を非推奨にする (#38)
* ignition起動用のパッケージを追加。メッシュファイルのパスが読み取れていない。

* ignition上にcrane_plusをspawnできた

* crane_plus_descriptionをigniotion用に改造

* ignitionに箱とテーブルを表示

* 箱を掴めるようにサンプルのパラメータ変更

* 依存パッケージを変更

* gazebo.materialスクリプトが読み込まれないため、パラメータを変更

* Dockerfile内でignitionのモデルをダウンロードする

* sunとground_planeもfuelからダウンロードする

* IgnitionとGazeboを共存させる

* Linterのチェックを通すための修正

* モデルのspawn位置を修正

* READMEのGazeboを使用する項目をIgnitionに置き換える

* 不要な変更を削除

File: crane_plus_description/urdf/crane_plus.gazebo.xacro (robot description, xacro)
@@ -1,4 +1,22 @@
 <?xml version="1.0"?>
 <robot xmlns:xacro="http://www.ros.org/wiki/xacro">
+  <xacro:macro name="material_gazebo_black">
+    <visual>
+      <material>
+        <ambient>0 0 0 1</ambient>
+        <diffuse>0 0 0 1</diffuse>
+        <specular>0.1 0.1 0.1 5.0</specular>
+      </material>
+    </visual>
+  </xacro:macro>
+  <xacro:macro name="material_gazebo_white">
+    <visual>
+      <material>
+        <ambient>1 1 1 1</ambient>
+        <diffuse>1 1 1 1</diffuse>
+        <specular>0.1 0.1 0.1 128.0</specular>
+      </material>
+    </visual>
+  </xacro:macro>
   <xacro:macro name="gazebo_robot_settings"
     params="name_link_base
@@ -7,40 +25,49 @@
             name_link_3
             name_link_4
-            name_link_hand">
+            name_link_hand
+            use_ignition
+            ">
     <gazebo>
-      <plugin filename="libgazebo_ros2_control.so" name="gazebo_ros2_control">
-        <robot_sim_type>gazebo_ros2_control/GazeboSystem</robot_sim_type>
-        <parameters>$(find crane_plus_control)/config/crane_plus_controllers.yaml</parameters>
-      </plugin>
+      <xacro:if value="${use_ignition}">
+        <plugin filename="libign_ros2_control-system.so" name="ign_ros2_control::IgnitionROS2ControlPlugin">
+          <parameters>$(find crane_plus_control)/config/crane_plus_controllers.yaml</parameters>
+        </plugin>
+      </xacro:if>
+      <xacro:unless value="${use_ignition}">
+        <plugin filename="libgazebo_ros2_control.so" name="gazebo_ros2_control">
+          <robot_sim_type>gazebo_ros2_control/GazeboSystem</robot_sim_type>
+          <parameters>$(find crane_plus_control)/config/crane_plus_controllers.yaml</parameters>
+        </plugin>
+      </xacro:unless>
     </gazebo>
     <gazebo reference="${name_link_base}">
       <mu1>0.2</mu1>
       <mu2>0.2</mu2>
-      <material>Gazebo/Black</material>
+      <xacro:material_gazebo_black/>
     </gazebo>
     <gazebo reference="${name_link_1}">
       <mu1>0.2</mu1>
       <mu2>0.2</mu2>
-      <material>Gazebo/White</material>
+      <xacro:material_gazebo_white/>
     </gazebo>
     <gazebo reference="${name_link_2}">
       <mu1>0.2</mu1>
       <mu2>0.2</mu2>
-      <material>Gazebo/Black</material>
+      <xacro:material_gazebo_black/>
     </gazebo>
     <gazebo reference="${name_link_3}">
       <mu1>0.2</mu1>
       <mu2>0.2</mu2>
-      <material>Gazebo/White</material>
+      <xacro:material_gazebo_white/>
     </gazebo>
     <gazebo reference="${name_link_4}">
       <mu1>0.2</mu1>
       <mu2>0.2</mu2>
-      <material>Gazebo/Black</material>
+      <xacro:material_gazebo_black/>
     </gazebo>
     <gazebo reference="${name_link_hand}">
       <mu1>0.2</mu1>
       <mu2>0.2</mu2>
-      <material>Gazebo/White</material>
+      <xacro:material_gazebo_white/>
     </gazebo>
   </xacro:macro>

File: crane_plus_description/urdf/crane_plus.gazebo_ros2_control.xacro (robot description, xacro)
@@ -17,8 +17,15 @@
             joint_4_upper_limit
             joint_hand_lower_limit
-            joint_hand_upper_limit">
+            joint_hand_upper_limit
+            use_ignition
+            ">
     <ros2_control name="${name}" type="system">
       <hardware>
-        <plugin>gazebo_ros2_control/GazeboSystem</plugin>
+        <xacro:if value="${use_ignition}">
+          <plugin>ign_ros2_control/IgnitionSystem</plugin>
+        </xacro:if>
+        <xacro:unless value="${use_ignition}">
+          <plugin>gazebo_ros2_control/GazeboSystem</plugin>
+        </xacro:unless>
       </hardware>
       <joint name="${name_joint_1}">

Commit message: カメラの画角調整

File: crane_plus_description/urdf/crane_plus.gazebo.xacro (robot description, xacro)
@@ -88,5 +88,5 @@
             <xacro:property name="camera_width" value="640"/>
             <xacro:property name="camera_height" value="480"/>
-            <xacro:property name="camera_hfov" value="${radians(120)}"/>
+            <xacro:property name="camera_hfov" value="${radians(70)}"/>
             <xacro:property name="camera_focal_length" value="${camera_width / (2 * tan(camera_hfov / 2))}"/>
             <horizontal_fov>${camera_hfov}</horizontal_fov>

Commit message: Gazebo環境にカメラを追加 (#83)
* カメラ追加

* use_sim_timeオプション追加

* カメラの画角調整

* 色検出サンプルの色しきい値調整

* 把持位置調整

* 現バージョンのデフォルト設定を反映

* ArUcoマーカ付きの立方体を追加

* ワールド、launchファイル追加

* use_cameraの有効化

* use_cameraを引数で切り替えられるように変更

* カメラスタンドのURDF修正

File: crane_plus_description/urdf/crane_plus.gazebo.xacro (robot description, xacro)
@@ -24,4 +24,5 @@
             name_link_4
             name_link_hand
+            use_camera
             use_ignition
             config_package
@@ -71,4 +72,52 @@
       <xacro:material_gazebo_white/>
     </gazebo>
+    <xacro:if value="$(arg use_camera)">
+      <gazebo>
+        <plugin filename="ignition-gazebo-sensors-system" name="ignition::gazebo::systems::Sensors">
+          <render_engine>ogre2</render_engine>
+        </plugin>
+      </gazebo>
+      <gazebo reference="camera_color_optical_frame">
+        <sensor name="camera" type="camera">
+          <pose relative_to="camera_color_optical_frame">0 0 0 ${radians(90)} ${radians(-90)} 0</pose>
+          <update_rate>10</update_rate>
+          <always_on>true</always_on>
+          <topic>image_raw</topic>
+          <gz_frame_id>camera_color_optical_frame</gz_frame_id>
+          <camera name="camera">
+            <xacro:property name="camera_width" value="640"/>
+            <xacro:property name="camera_height" value="480"/>
+            <xacro:property name="camera_hfov" value="${radians(70)}"/>
+            <xacro:property name="camera_focal_length" value="${camera_width / (2 * tan(camera_hfov / 2))}"/>
+            <horizontal_fov>${camera_hfov}</horizontal_fov>
+            <image>
+              <width>${camera_width}</width>
+              <height>${camera_height}</height>
+            </image>
+            <clip>
+              <near>0.1</near>
+              <far>10.0</far>
+            </clip>
+            <lens>
+              <intrinsics>
+                <fx>${camera_focal_length}</fx>
+                <fy>${camera_focal_length}</fy>
+                <cx>${(camera_width + 1) / 2}</cx>
+                <cy>${(camera_height + 1) / 2}</cy>
+                <s>1.0</s>
+              </intrinsics>
+              <projection>
+                <p_fx>${camera_focal_length}</p_fx>
+                <p_fy>${camera_focal_length}</p_fy>
+                <p_cx>${(camera_width + 1) / 2}</p_cx>
+                <p_cy>${(camera_height + 1) / 2}</p_cy>
+                <tx>0</tx>
+                <ty>0</ty>
+              </projection>
+            </lens>
+          </camera>
+        </sensor>
+      </gazebo>
+    </xacro:if>
   </xacro:macro>
 </robot>

Commit message: Gazebo環境にカメラを追加 (#83)
* カメラ追加

* use_sim_timeオプション追加

* カメラの画角調整

* 色検出サンプルの色しきい値調整

* 把持位置調整

* 現バージョンのデフォルト設定を反映

* ArUcoマーカ付きの立方体を追加

* ワールド、launchファイル追加

* use_cameraの有効化

* use_cameraを引数で切り替えられるように変更

* カメラスタンドのURDF修正

File: crane_plus_description/urdf/crane_plus.gazebo.xacro (robot description, xacro)
@@ -24,4 +24,6 @@
             name_link_4
             name_link_hand
+            use_camera
+            use_ignition
             config_package
             config_file_path
@@ -62,4 +64,52 @@
       <xacro:material_gazebo_white/>
     </gazebo>
+    <xacro:if value="$(arg use_camera)">
+      <gazebo>
+        <plugin filename="ignition-gazebo-sensors-system" name="ignition::gazebo::systems::Sensors">
+          <render_engine>ogre2</render_engine>
+        </plugin>
+      </gazebo>
+      <gazebo reference="camera_color_optical_frame">
+        <sensor name="camera" type="camera">
+          <pose relative_to="camera_color_optical_frame">0 0 0 ${radians(90)} ${radians(-90)} 0</pose>
+          <update_rate>10</update_rate>
+          <always_on>true</always_on>
+          <topic>image_raw</topic>
+          <gz_frame_id>camera_color_optical_frame</gz_frame_id>
+          <camera name="camera">
+            <xacro:property name="camera_width" value="640"/>
+            <xacro:property name="camera_height" value="480"/>
+            <xacro:property name="camera_hfov" value="${radians(70)}"/>
+            <xacro:property name="camera_focal_length" value="${camera_width / (2 * tan(camera_hfov / 2))}"/>
+            <horizontal_fov>${camera_hfov}</horizontal_fov>
+            <image>
+              <width>${camera_width}</width>
+              <height>${camera_height}</height>
+            </image>
+            <clip>
+              <near>0.1</near>
+              <far>10.0</far>
+            </clip>
+            <lens>
+              <intrinsics>
+                <fx>${camera_focal_length}</fx>
+                <fy>${camera_focal_length}</fy>
+                <cx>${(camera_width + 1) / 2}</cx>
+                <cy>${(camera_height + 1) / 2}</cy>
+                <s>1.0</s>
+              </intrinsics>
+              <projection>
+                <p_fx>${camera_focal_length}</p_fx>
+                <p_fy>${camera_focal_length}</p_fy>
+                <p_cx>${(camera_width + 1) / 2}</p_cx>
+                <p_cy>${(camera_height + 1) / 2}</p_cy>
+                <tx>0</tx>
+                <ty>0</ty>
+              </projection>
+            </lens>
+          </camera>
+        </sensor>
+      </gazebo>
+    </xacro:if>
   </xacro:macro>
 </robot>

File: crane_plus_description/urdf/crane_plus.urdf.xacro (robot description, xacro)
@@ -117,4 +117,6 @@
       name_link_4="${NAME_LINK_4}"
       name_link_hand="${NAME_LINK_HAND}"
+      use_camera="$(arg use_camera)"
+      use_ignition="$(arg use_ignition)"
       config_package="$(arg gz_control_config_package)"
       config_file_path="$(arg gz_control_config_file_path)" />

Commit message: gazebo_robot_settingsマクロのパラメータを削除

File: crane_plus_description/urdf/crane_plus.gazebo.xacro (robot description, xacro)
@@ -17,51 +17,41 @@
     </visual>
   </xacro:macro>
-  <xacro:macro name="gazebo_robot_settings"
-    params="name_link_base
-            name_link_1
-            name_link_2
-            name_link_3
-            name_link_4
-            name_link_hand
-            use_camera
-            config_package
-            config_file_path
-            ">
+  <xacro:macro name="gazebo_robot_settings">
     <gazebo>
       <plugin filename="libgz_ros2_control-system.so" name="gz_ros2_control::GazeboSimROS2ControlPlugin">
-      <parameters>$(find ${config_package})/${config_file_path}</parameters>
+      <parameters>$(find ${GZ_CONTROL_CONFIG_PACKAGE})/${GZ_CONTROL_CONFIG_FILE_PATH}</parameters>
       </plugin>
     </gazebo>
-    <gazebo reference="${name_link_base}">
+    <gazebo reference="${NAME_LINK_BASE}">
       <mu1>0.2</mu1>
       <mu2>0.2</mu2>
       <xacro:material_gazebo_black/>
     </gazebo>
-    <gazebo reference="${name_link_1}">
+    <gazebo reference="${NAME_LINK_1}">
       <mu1>0.2</mu1>
       <mu2>0.2</mu2>
       <xacro:material_gazebo_white/>
     </gazebo>
-    <gazebo reference="${name_link_2}">
+    <gazebo reference="${NAME_LINK_2}">
       <mu1>0.2</mu1>
       <mu2>0.2</mu2>
       <xacro:material_gazebo_black/>
     </gazebo>
-    <gazebo reference="${name_link_3}">
+    <gazebo reference="${NAME_LINK_3}">
       <mu1>0.2</mu1>
       <mu2>0.2</mu2>
       <xacro:material_gazebo_white/>
     </gazebo>
-    <gazebo reference="${name_link_4}">
+    <gazebo reference="${NAME_LINK_4}">
       <mu1>0.2</mu1>
       <mu2>0.2</mu2>
       <xacro:material_gazebo_black/>
     </gazebo>
-    <gazebo reference="${name_link_hand}">
+    <gazebo reference="${NAME_LINK_HAND}">
       <mu1>0.2</mu1>
       <mu2>0.2</mu2>
       <xacro:material_gazebo_white/>
     </gazebo>
-    <xacro:if value="$(arg use_camera)">
+    <xacro:if value="${USE_CAMERA}">
       <gazebo>
           <plugin filename="gz-sim-sensors-system" name="gz::sim::systems::Sensors">

File: crane_plus_description/urdf/crane_plus.urdf.xacro (robot description, xacro)
@@ -17,4 +17,7 @@
   <xacro:arg name="gz_control_config_package" default="" />
   <xacro:arg name="gz_control_config_file_path" default="" />
+  <xacro:property name="USE_CAMERA" value="$(arg use_camera)"/>
+  <xacro:property name="GZ_CONTROL_CONFIG_PACKAGE" value="$(arg gz_control_config_package)"/>
+  <xacro:property name="GZ_CONTROL_CONFIG_FILE_PATH" value="$(arg gz_control_config_file_path)"/>
   <xacro:property name="NAME_LINK_BASE" value="crane_plus_base"/>
   <xacro:property name="NAME_LINK_1" value="crane_plus_link1"/>
@@ -81,14 +84,5 @@
   </xacro:unless>
   <xacro:if value="$(arg use_gazebo)">
-    <xacro:gazebo_robot_settings
-      name_link_base="${NAME_LINK_BASE}"
-      name_link_1="${NAME_LINK_1}"
-      name_link_2="${NAME_LINK_2}"
-      name_link_3="${NAME_LINK_3}"
-      name_link_4="${NAME_LINK_4}"
-      name_link_hand="${NAME_LINK_HAND}"
-      use_camera="$(arg use_camera)"
-      config_package="$(arg gz_control_config_package)"
-      config_file_path="$(arg gz_control_config_file_path)" />
+    <xacro:gazebo_robot_settings />
     <xacro:crane_plus_gazebo_ros2_control_settings
       name="crane_plus"
