Commit message: リンク名とジョイント名のpropertyを廃止

File: crane_plus_description/urdf/crane_plus.gazebo.xacro (robot description, xacro)
@@ -23,30 +23,30 @@
       </plugin>
     </gazebo>
-    <gazebo reference="${NAME_LINK_BASE}">
+    <gazebo reference="crane_plus_base">
       <mu1>0.2</mu1>
       <mu2>0.2</mu2>
       <xacro:material_gazebo_black/>
     </gazebo>
-    <gazebo reference="${NAME_LINK_1}">
+    <gazebo reference="crane_plus_link1">
       <mu1>0.2</mu1>
       <mu2>0.2</mu2>
       <xacro:material_gazebo_white/>
     </gazebo>
-    <gazebo reference="${NAME_LINK_2}">
+    <gazebo reference="crane_plus_link2">
       <mu1>0.2</mu1>
       <mu2>0.2</mu2>
       <xacro:material_gazebo_black/>
     </gazebo>
-    <gazebo reference="${NAME_LINK_3}">
+    <gazebo reference="crane_plus_link3">
       <mu1>0.2</mu1>
       <mu2>0.2</mu2>
       <xacro:material_gazebo_white/>
     </gazebo>
-    <gazebo reference="${NAME_LINK_4}">
+    <gazebo reference="crane_plus_link4">
       <mu1>0.2</mu1>
       <mu2>0.2</mu2>
       <xacro:material_gazebo_black/>
     </gazebo>
-    <gazebo reference="${NAME_LINK_HAND}">
+    <gazebo reference="crane_plus_link_hand">
       <mu1>0.2</mu1>
       <mu2>0.2</mu2>

File: crane_plus_description/urdf/crane_plus.gazebo_ros2_control.xacro (robot description, xacro)
@@ -6,5 +6,5 @@
         <plugin>gz_ros2_control/GazeboSimSystem</plugin>
       </hardware>
-      <joint name="${NAME_JOINT_1}">
+      <joint name="crane_plus_joint1">
         <command_interface name="position">
           <param name="min">${JOINT_1_LOWER_LIMIT}</param>
@@ -15,5 +15,5 @@
         <state_interface name="effort"/>
       </joint>
-      <joint name="${NAME_JOINT_2}">
+      <joint name="crane_plus_joint2">
         <command_interface name="position">
           <param name="min">${JOINT_2_LOWER_LIMIT}</param>
@@ -24,5 +24,5 @@
         <state_interface name="effort"/>
       </joint>
-      <joint name="${NAME_JOINT_3}">
+      <joint name="crane_plus_joint3">
         <command_interface name="position">
           <param name="min">${JOINT_3_LOWER_LIMIT}</param>
@@ -33,5 +33,5 @@
         <state_interface name="effort"/>
       </joint>
-      <joint name="${NAME_JOINT_4}">
+      <joint name="crane_plus_joint4">
         <command_interface name="position">
           <param name="min">${JOINT_4_LOWER_LIMIT}</param>
@@ -42,5 +42,5 @@
         <state_interface name="effort"/>
       </joint>
-      <joint name="${NAME_JOINT_HAND}">
+      <joint name="crane_plus_joint_hand">
         <command_interface name="position">
           <param name="min">${JOINT_HAND_LOWER_LIMIT}</param>

File: crane_plus_description/urdf/crane_plus.ros2_control.xacro (robot description, xacro)
@@ -18,5 +18,5 @@
         </xacro:unless>
       </hardware>
-      <joint name="${NAME_JOINT_1}">
+      <joint name="crane_plus_joint1">
         <command_interface name="position">
           <param name="min">${JOINT_1_LOWER_LIMIT}</param>
@@ -30,5 +30,5 @@
         <param name="dxl_id">1</param>
       </joint>
-      <joint name="${NAME_JOINT_2}">
+      <joint name="crane_plus_joint2">
         <command_interface name="position">
           <param name="min">${JOINT_2_LOWER_LIMIT}</param>
@@ -42,5 +42,5 @@
         <param name="dxl_id">2</param>
       </joint>
-      <joint name="${NAME_JOINT_3}">
+      <joint name="crane_plus_joint3">
         <command_interface name="position">
           <param name="min">${JOINT_3_LOWER_LIMIT}</param>
@@ -54,5 +54,5 @@
         <param name="dxl_id">3</param>
       </joint>
-      <joint name="${NAME_JOINT_4}">
+      <joint name="crane_plus_joint4">
         <command_interface name="position">
           <param name="min">${JOINT_4_LOWER_LIMIT}</param>
@@ -66,5 +66,5 @@
         <param name="dxl_id">4</param>
       </joint>
-      <joint name="${NAME_JOINT_HAND}">
+      <joint name="crane_plus_joint_hand">
         <command_interface name="position">
           <param name="min">${JOINT_HAND_LOWER_LIMIT}</param>

File: crane_plus_description/urdf/crane_plus.urdf.xacro (robot description, xacro)
@@ -37,18 +37,4 @@
     <color rgba="0.8 0.8 0.8 1.0" />
   </material>
-  <xacro:property name="NAME_LINK_BASE" value="crane_plus_base"/>
-  <xacro:property name="NAME_LINK_1" value="crane_plus_link1"/>
-  <xacro:property name="NAME_LINK_2" value="crane_plus_link2"/>
-  <xacro:property name="NAME_LINK_3" value="crane_plus_link3"/>
-  <xacro:property name="NAME_LINK_4" value="crane_plus_link4"/>
-  <xacro:property name="NAME_LINK_HAND" value="crane_plus_link_hand"/>
-  <xacro:property name="NAME_LINK_TCP" value="crane_plus_link_tcp"/>
-  <xacro:property name="NAME_JOINT_BASE" value="crane_plus_joint_base"/>
-  <xacro:property name="NAME_JOINT_1" value="crane_plus_joint1"/>
-  <xacro:property name="NAME_JOINT_2" value="crane_plus_joint2"/>
-  <xacro:property name="NAME_JOINT_3" value="crane_plus_joint3"/>
-  <xacro:property name="NAME_JOINT_4" value="crane_plus_joint4"/>
-  <xacro:property name="NAME_JOINT_HAND" value="crane_plus_joint_hand"/>
-  <xacro:property name="NAME_JOINT_TCP" value="crane_plus_joint_tcp"/>
   <xacro:property name="SERVO_HOME" value="${radians(150.0)}"/>
   <xacro:property name="JOINT_EFFORT_LIMIT" value="1.5"/>
@@ -84,6 +70,6 @@
     <xacro:include filename="$(find crane_plus_description)/urdf/camera.xacro" />
     <xacro:include filename="$(find crane_plus_description)/urdf/camera_stand.xacro" />
-    <xacro:sensor_camera parent="${NAME_LINK_BASE}" />
-    <xacro:camera_stand parent="${NAME_LINK_BASE}" />
+    <xacro:sensor_camera parent="crane_plus_base" />
+    <xacro:camera_stand parent="crane_plus_base" />
   </xacro:if>
 </robot>

File: crane_plus_description/urdf/crane_plus.xacro (robot description, xacro)
@@ -2,10 +2,10 @@
 <robot xmlns:xacro="http://ros.org/wiki/xacro">
   <xacro:macro name="crane_plus" params="parent *origin">
-    <joint name="${NAME_JOINT_BASE}" type="fixed">
+    <joint name="crane_plus_joint_base" type="fixed">
       <xacro:insert_block name="origin"/>
       <parent link="${parent}"/>
-      <child link="${NAME_LINK_BASE}"/>
-    </joint>
-    <link name="${NAME_LINK_BASE}">
+      <child link="crane_plus_base"/>
+    </joint>
+    <link name="crane_plus_base">
       <visual>
         <origin xyz="0 0 0" rpy="0 0 0"/>
@@ -28,5 +28,5 @@
       </inertial>
     </link>
-    <joint name="${NAME_JOINT_1}" type="revolute">
+    <joint name="crane_plus_joint1" type="revolute">
       <origin xyz="0 0 0.0454" rpy="0 0 0"/>
       <axis xyz="0 0 1"/>
@@ -37,9 +37,9 @@
         upper="${JOINT_1_UPPER_LIMIT}"
         />
-      <parent link="${NAME_LINK_BASE}"/>
-      <child link="${NAME_LINK_1}"/>
-      <dynamics damping="1.0e-6" friction="2.0e-1"/>
-    </joint>
-    <link name="${NAME_LINK_1}">
+      <parent link="crane_plus_base"/>
+      <child link="crane_plus_link1"/>
+      <dynamics damping="1.0e-6" friction="2.0e-1"/>
+    </joint>
+    <link name="crane_plus_link1">
       <visual>
         <origin xyz="0 0 0" rpy="0 0 0"/>
@@ -62,5 +62,5 @@
       </inertial>
     </link>
-    <joint name="${NAME_JOINT_2}" type="revolute">
+    <joint name="crane_plus_joint2" type="revolute">
       <origin xyz="0 0 0.026" rpy="0 0 0"/>
       <axis xyz="0 1 0"/>
@@ -71,9 +71,9 @@
         upper="${JOINT_2_UPPER_LIMIT}"
         />
-      <parent link="${NAME_LINK_1}"/>
-      <child link="${NAME_LINK_2}"/>
-      <dynamics damping="1.0e-6" friction="2.0e-1"/>
-    </joint>
-    <link name="${NAME_LINK_2}">
+      <parent link="crane_plus_link1"/>
+      <child link="crane_plus_link2"/>
+      <dynamics damping="1.0e-6" friction="2.0e-1"/>
+    </joint>
+    <link name="crane_plus_link2">
       <visual>
         <origin xyz="0 0 0" rpy="${radians(90)} 0 0"/>
@@ -96,5 +96,5 @@
       </inertial>
     </link>
-    <joint name="${NAME_JOINT_3}" type="revolute">
+    <joint name="crane_plus_joint3" type="revolute">
       <origin xyz="0 0 0.083" rpy="0 0 0"/>
       <axis xyz="0 -1 0"/>
@@ -105,9 +105,9 @@
         upper="${JOINT_3_UPPER_LIMIT}"
         />
-      <parent link="${NAME_LINK_2}"/>
-      <child link="${NAME_LINK_3}"/>
-      <dynamics damping="1.0e-6" friction="2.0e-1"/>
-    </joint>
-    <link name="${NAME_LINK_3}">
+      <parent link="crane_plus_link2"/>
+      <child link="crane_plus_link3"/>
+      <dynamics damping="1.0e-6" friction="2.0e-1"/>
+    </joint>
+    <link name="crane_plus_link3">
       <visual>
         <origin xyz="0 0 0" rpy="${radians(90)} 0 0"/>
@@ -130,5 +130,5 @@
       </inertial>
     </link>
-    <joint name="${NAME_JOINT_4}" type="revolute">
+    <joint name="crane_plus_joint4" type="revolute">
       <origin xyz="0 0 0.0935" rpy="0 0 0"/>
       <axis xyz="0 -1 0"/>
@@ -139,9 +139,9 @@
         upper="${JOINT_4_UPPER_LIMIT}"
         />
-      <parent link="${NAME_LINK_3}"/>
-      <child link="${NAME_LINK_4}"/>
-      <dynamics damping="1.0e-6" friction="2.0e-1"/>
-    </joint>
-    <link name="${NAME_LINK_4}">
+      <parent link="crane_plus_link3"/>
+      <child link="crane_plus_link4"/>
+      <dynamics damping="1.0e-6" friction="2.0e-1"/>
+    </joint>
+    <link name="crane_plus_link4">
       <visual>
         <origin xyz="0 0 0" rpy="${radians(90)} 0 0"/>
@@ -164,5 +164,5 @@
       </inertial>
     </link>
-    <joint name="${NAME_JOINT_HAND}" type="revolute">
+    <joint name="crane_plus_joint_hand" type="revolute">
       <origin xyz="0 -0.0145 0.045" rpy="0 0 0"/>
       <axis xyz="-1 0 0"/>
@@ -173,9 +173,9 @@
         upper="${JOINT_HAND_UPPER_LIMIT}"
         />
-      <parent link="${NAME_LINK_4}"/>
-      <child link="${NAME_LINK_HAND}"/>
-      <dynamics damping="1.0e-6" friction="2.0e-1"/>
-    </joint>
-    <link name="${NAME_LINK_HAND}">
+      <parent link="crane_plus_link4"/>
+      <child link="crane_plus_link_hand"/>
+      <dynamics damping="1.0e-6" friction="2.0e-1"/>
+    </joint>
+    <link name="crane_plus_link_hand">
       <visual>
         <origin xyz="0 0 0" rpy="0 ${radians(-90)} 0"/>
@@ -198,10 +198,10 @@
       </inertial>
     </link>
-    <joint name="${NAME_JOINT_TCP}" type="fixed">
+    <joint name="crane_plus_joint_tcp" type="fixed">
       <origin xyz="0 0 0.121" rpy="0 0 0"/>
-      <parent link="${NAME_LINK_4}"/>
-      <child link="${NAME_LINK_TCP}"/>
-    </joint>
-    <link name="${NAME_LINK_TCP}"/>
+      <parent link="crane_plus_link4"/>
+      <child link="crane_plus_link_tcp"/>
+    </joint>
+    <link name="crane_plus_link_tcp"/>
   </xacro:macro>
 </robot>

Commit message: 引数のpropertyを廃止

File: crane_plus_description/urdf/crane_plus.gazebo.xacro (robot description, xacro)
@@ -17,8 +17,8 @@
     </visual>
   </xacro:macro>
-  <xacro:macro name="gazebo_robot_settings">
+  <xacro:macro name="gazebo_robot_settings" params="use_camera gz_control_config_package gz_control_config_file_path">
     <gazebo>
       <plugin filename="libgz_ros2_control-system.so" name="gz_ros2_control::GazeboSimROS2ControlPlugin">
-      <parameters>$(find ${GZ_CONTROL_CONFIG_PACKAGE})/${GZ_CONTROL_CONFIG_FILE_PATH}</parameters>
+      <parameters>$(find ${gz_control_config_package})/${gz_control_config_file_path}</parameters>
       </plugin>
     </gazebo>
@@ -53,5 +53,5 @@
       <xacro:material_gazebo_white/>
     </gazebo>
-    <xacro:if value="${USE_CAMERA}">
+    <xacro:if value="${use_camera}">
       <gazebo>
           <plugin filename="gz-sim-sensors-system" name="gz::sim::systems::Sensors">

File: crane_plus_description/urdf/crane_plus.ros2_control.xacro (robot description, xacro)
@@ -1,19 +1,21 @@
 <?xml version="1.0"?>
 <robot xmlns:xacro="http://www.ros.org/wiki/xacro">
-  <xacro:macro name="crane_plus_ros2_control_settings">
+  <xacro:macro name="crane_plus_ros2_control_settings"
+    params="use_mock_components port_name baudrate timeout_seconds
+            read_velocities read_loads read_voltages read_temperatures">
     <ros2_control name="crane_plus" type="system">
       <hardware>
-        <xacro:if value="${USE_MOCK_COMPONENTS}">
+        <xacro:if value="${use_mock_components}">
           <plugin>mock_components/GenericSystem</plugin>
         </xacro:if>
-        <xacro:unless value="${USE_MOCK_COMPONENTS}">
+        <xacro:unless value="${use_mock_components}">
           <plugin>crane_plus_hardware/CranePlusHardware</plugin>
-          <param name="port_name">${PORT_NAME}</param>
-          <param name="baudrate">${BAUDRATE}</param>
-          <param name="timeout_seconds">${TIMEOUT_SECONDS}</param>
-          <param name="read_velocities">${READ_VELOCITIES}</param>
-          <param name="read_loads">${READ_LOADS}</param>
-          <param name="read_voltages">${READ_VOLTAGES}</param>
-          <param name="read_temperatures">${READ_TEMPERATURES}</param>
+          <param name="port_name">${port_name}</param>
+          <param name="baudrate">${baudrate}</param>
+          <param name="timeout_seconds">${timeout_seconds}</param>
+          <param name="read_velocities">${read_velocities}</param>
+          <param name="read_loads">${read_loads}</param>
+          <param name="read_voltages">${read_voltages}</param>
+          <param name="read_temperatures">${read_temperatures}</param>
         </xacro:unless>
       </hardware>

File: crane_plus_description/urdf/crane_plus.urdf.xacro (robot description, xacro)
@@ -17,15 +17,4 @@
   <xacro:arg name="gz_control_config_package" default="" />
   <xacro:arg name="gz_control_config_file_path" default="" />
-  <xacro:property name="USE_CAMERA" value="$(arg use_camera)"/>
-  <xacro:property name="USE_MOCK_COMPONENTS" value="$(arg use_mock_components)"/>
-  <xacro:property name="PORT_NAME" value="$(arg port_name)"/>
-  <xacro:property name="BAUDRATE" value="$(arg baudrate)"/>
-  <xacro:property name="TIMEOUT_SECONDS" value="$(arg timeout_seconds)"/>
-  <xacro:property name="READ_VELOCITIES" value="$(arg read_velocities)"/>
-  <xacro:property name="READ_LOADS" value="$(arg read_loads)"/>
-  <xacro:property name="READ_VOLTAGES" value="$(arg read_voltages)"/>
-  <xacro:property name="READ_TEMPERATURES" value="$(arg read_temperatures)"/>
-  <xacro:property name="GZ_CONTROL_CONFIG_PACKAGE" value="$(arg gz_control_config_package)"/>
-  <xacro:property name="GZ_CONTROL_CONFIG_FILE_PATH" value="$(arg gz_control_config_file_path)"/>
   <material name="black">
     <color rgba="0.2 0.2 0.2 1.0"/>
@@ -61,8 +50,21 @@
   </xacro:crane_plus>
   <xacro:unless value="$(arg use_gazebo)">
-    <xacro:crane_plus_ros2_control_settings />
+    <xacro:crane_plus_ros2_control_settings
+      use_mock_components="$(arg use_mock_components)"
+      port_name="$(arg port_name)"
+      baudrate="$(arg baudrate)"
+      timeout_seconds="$(arg timeout_seconds)"
+      read_velocities="$(arg read_velocities)"
+      read_loads="$(arg read_loads)"
+      read_voltages="$(arg read_voltages)"
+      read_temperatures="$(arg read_temperatures)"
+      />
   </xacro:unless>
   <xacro:if value="$(arg use_gazebo)">
-    <xacro:gazebo_robot_settings />
+    <xacro:gazebo_robot_settings
+      use_camera="$(arg use_camera)"
+      gz_control_config_package="$(arg gz_control_config_package)"
+      gz_control_config_file_path="$(arg gz_control_config_file_path)"
+      />
     <xacro:crane_plus_gazebo_ros2_control_settings />
   </xacro:if>
