Commit message: 不要なpropertyを廃止 (#98)
* リンク名とジョイント名のpropertyを廃止

* 引数のpropertyを廃止

File: crane_plus_description/urdf/crane_plus.gazebo.xacro (robot description, xacro)
@@ -17,41 +17,41 @@
     </visual>
   </xacro:macro>
-  <xacro:macro name="gazebo_robot_settings">
+  <xacro:macro name="gazebo_robot_settings" params="use_camera gz_control_config_package gz_control_config_file_path">
     <gazebo>
       <plugin filename="libgz_ros2_control-system.so" name="gz_ros2_control::GazeboSimROS2ControlPlugin">
-      <parameters>$(find ${GZ_CONTROL_CONFIG_PACKAGE})/${GZ_CONTROL_CONFIG_FILE_PATH}</parameters>
+      <parameters>$(find ${gz_control_config_package})/${gz_control_config_file_path}</parameters>
       </plugin>
     </gazebo>
-    <gazebo reference="${NAME_LINK_BASE}">
+    <gazebo reference="crane_plus_base">
       <mu1>0.2</mu1>
       <mu2>0.2</mu2>
       <xacro:material_gazebo_black/>
     </gazebo>
-    <gazebo reference="${NAME_LINK_1}">
+    <gazebo reference="crane_plus_link1">
       <mu1>0.2</mu1>
       <mu2>0.2</mu2>
       <xacro:material_gazebo_white/>
     </gazebo>
-    <gazebo reference="${NAME_LINK_2}">
+    <gazebo reference="crane_plus_link2">
       <mu1>0.2</mu1>
       <mu2>0.2</mu2>
       <xacro:material_gazebo_black/>
     </gazebo>
-    <gazebo reference="${NAME_LINK_3}">
+    <gazebo reference="crane_plus_link3">
       <mu1>0.2</mu1>
       <mu2>0.2</mu2>
       <xacro:material_gazebo_white/>
     </gazebo>
-    <gazebo reference="${NAME_LINK_4}">
+    <gazebo reference="crane_plus_link4">
       <mu1>0.2</mu1>
       <mu2>0.2</mu2>
       <xacro:material_gazebo_black/>
     </gazebo>
-    <gazebo reference="${NAME_LINK_HAND}">
+    <gazebo reference="crane_plus_link_hand">
       <mu1>0.2</mu1>
       <mu2>0.2</mu2>
       <xacro:material_gazebo_white/>
     </gazebo>
-    <xacro:if value="${USE_CAMERA}">
+    <xacro:if value="${use_camera}">
       <gazebo>
           <plugin filename="gz-sim-sensors-system" name="gz::sim::systems::Sensors">

File: crane_plus_description/urdf/crane_plus.ros2_control.xacro (robot description, xacro)
@@ -1,22 +1,24 @@
 <?xml version="1.0"?>
 <robot xmlns:xacro="http://www.ros.org/wiki/xacro">
-  <xacro:macro name="crane_plus_ros2_control_settings">
+  <xacro:macro name="crane_plus_ros2_control_settings"
+    params="use_mock_components port_name baudrate timeout_seconds
+            read_velocities read_loads read_voltages read_temperatures">
     <ros2_control name="crane_plus" type="system">
       <hardware>
-        <xacro:if value="${USE_MOCK_COMPONENTS}">
+        <xacro:if value="${use_mock_components}">
           <plugin>mock_components/GenericSystem</plugin>
         </xacro:if>
-        <xacro:unless value="${USE_MOCK_COMPONENTS}">
+        <xacro:unless value="${use_mock_components}">
           <plugin>crane_plus_hardware/CranePlusHardware</plugin>
-          <param name="port_name">${PORT_NAME}</param>
-          <param name="baudrate">${BAUDRATE}</param>
-          <param name="timeout_seconds">${TIMEOUT_SECONDS}</param>
-          <param name="read_velocities">${READ_VELOCITIES}</param>
-          <param name="read_loads">${READ_LOADS}</param>
-          <param name="read_voltages">${READ_VOLTAGES}</param>
-          <param name="read_temperatures">${READ_TEMPERATURES}</param>
+          <param name="port_name">${port_name}</param>
+          <param name="baudrate">${baudrate}</param>
+          <param name="timeout_seconds">${timeout_seconds}</param>
+          <param name="read_velocities">${read_velocities}</param>
+          <param name="read_loads">${read_loads}</param>
+          <param name="read_voltages">${read_voltages}</param>
+          <param name="read_temperatures">${read_temperatures}</param>
         </xacro:unless>
       </hardware>
-      <joint name="${NAME_JOINT_1}">
+      <joint name="crane_plus_joint1">
         <command_interface name="position">
           <param name="min">${JOINT_1_LOWER_LIMIT}</param>
@@ -30,5 +32,5 @@
         <param name="dxl_id">1</param>
       </joint>
-      <joint name="${NAME_JOINT_2}">
+      <joint name="crane_plus_joint2">
         <command_interface name="position">
           <param name="min">${JOINT_2_LOWER_LIMIT}</param>
@@ -42,5 +44,5 @@
         <param name="dxl_id">2</param>
       </joint>
-      <joint name="${NAME_JOINT_3}">
+      <joint name="crane_plus_joint3">
         <command_interface name="position">
           <param name="min">${JOINT_3_LOWER_LIMIT}</param>
@@ -54,5 +56,5 @@
         <param name="dxl_id">3</param>
       </joint>
-      <joint name="${NAME_JOINT_4}">
+      <joint name="crane_plus_joint4">
         <command_interface name="position">
           <param name="min">${JOINT_4_LOWER_LIMIT}</param>
@@ -66,5 +68,5 @@
         <param name="dxl_id">4</param>
       </joint>
-      <joint name="${NAME_JOINT_HAND}">
+      <joint name="crane_plus_joint_hand">
         <command_interface name="position">
           <param name="min">${JOINT_HAND_LOWER_LIMIT}</param>

File: crane_plus_description/urdf/crane_plus.urdf.xacro (robot description, xacro)
@@ -17,15 +17,4 @@
   <xacro:arg name="gz_control_config_package" default="" />
   <xacro:arg name="gz_control_config_file_path" default="" />
-  <xacro:property name="USE_CAMERA" value="$(arg use_camera)"/>
-  <xacro:property name="USE_MOCK_COMPONENTS" value="$(arg use_mock_components)"/>
-  <xacro:property name="PORT_NAME" value="$(arg port_name)"/>
-  <xacro:property name="BAUDRATE" value="$(arg baudrate)"/>
-  <xacro:property name="TIMEOUT_SECONDS" value="$(arg timeout_seconds)"/>
-  <xacro:property name="READ_VELOCITIES" value="$(arg read_velocities)"/>
-  <xacro:property name="READ_LOADS" value="$(arg read_loads)"/>
-  <xacro:property name="READ_VOLTAGES" value="$(arg read_voltages)"/>
-  <xacro:property name="READ_TEMPERATURES" value="$(arg read_temperatures)"/>
-  <xacro:property name="GZ_CONTROL_CONFIG_PACKAGE" value="$(arg gz_control_config_package)"/>
-  <xacro:property name="GZ_CONTROL_CONFIG_FILE_PATH" value="$(arg gz_control_config_file_path)"/>
   <material name="black">
     <color rgba="0.2 0.2 0.2 1.0"/>
@@ -37,18 +26,4 @@
     <color rgba="0.8 0.8 0.8 1.0" />
   </material>
-  <xacro:property name="NAME_LINK_BASE" value="crane_plus_base"/>
-  <xacro:property name="NAME_LINK_1" value="crane_plus_link1"/>
-  <xacro:property name="NAME_LINK_2" value="crane_plus_link2"/>
-  <xacro:property name="NAME_LINK_3" value="crane_plus_link3"/>
-  <xacro:property name="NAME_LINK_4" value="crane_plus_link4"/>
-  <xacro:property name="NAME_LINK_HAND" value="crane_plus_link_hand"/>
-  <xacro:property name="NAME_LINK_TCP" value="crane_plus_link_tcp"/>
-  <xacro:property name="NAME_JOINT_BASE" value="crane_plus_joint_base"/>
-  <xacro:property name="NAME_JOINT_1" value="crane_plus_joint1"/>
-  <xacro:property name="NAME_JOINT_2" value="crane_plus_joint2"/>
-  <xacro:property name="NAME_JOINT_3" value="crane_plus_joint3"/>
-  <xacro:property name="NAME_JOINT_4" value="crane_plus_joint4"/>
-  <xacro:property name="NAME_JOINT_HAND" value="crane_plus_joint_hand"/>
-  <xacro:property name="NAME_JOINT_TCP" value="crane_plus_joint_tcp"/>
   <xacro:property name="SERVO_HOME" value="${radians(150.0)}"/>
   <xacro:property name="JOINT_EFFORT_LIMIT" value="1.5"/>
@@ -75,8 +50,21 @@
   </xacro:crane_plus>
   <xacro:unless value="$(arg use_gazebo)">
-    <xacro:crane_plus_ros2_control_settings />
+    <xacro:crane_plus_ros2_control_settings
+      use_mock_components="$(arg use_mock_components)"
+      port_name="$(arg port_name)"
+      baudrate="$(arg baudrate)"
+      timeout_seconds="$(arg timeout_seconds)"
+      read_velocities="$(arg read_velocities)"
+      read_loads="$(arg read_loads)"
+      read_voltages="$(arg read_voltages)"
+      read_temperatures="$(arg read_temperatures)"
+      />
   </xacro:unless>
   <xacro:if value="$(arg use_gazebo)">
-    <xacro:gazebo_robot_settings />
+    <xacro:gazebo_robot_settings
+      use_camera="$(arg use_camera)"
+      gz_control_config_package="$(arg gz_control_config_package)"
+      gz_control_config_file_path="$(arg gz_control_config_file_path)"
+      />
     <xacro:crane_plus_gazebo_ros2_control_settings />
   </xacro:if>
@@ -84,6 +72,6 @@
     <xacro:include filename="$(find crane_plus_description)/urdf/camera.xacro" />
     <xacro:include filename="$(find crane_plus_description)/urdf/camera_stand.xacro" />
-    <xacro:sensor_camera parent="${NAME_LINK_BASE}" />
-    <xacro:camera_stand parent="${NAME_LINK_BASE}" />
+    <xacro:sensor_camera parent="crane_plus_base" />
+    <xacro:camera_stand parent="crane_plus_base" />
   </xacro:if>
 </robot>
