Commit message: crane_plus_ros2_control_settingsマクロのパラメータを削除

File: crane_plus_description/urdf/crane_plus.ros2_control.xacro (robot description, xacro)
@@ -1,49 +1,25 @@
 <?xml version="1.0"?>
 <robot xmlns:xacro="http://www.ros.org/wiki/xacro">
-  <xacro:macro name="crane_plus_ros2_control_settings"
-    params="name
-            name_joint_1
-            name_joint_2
-            name_joint_3
-            name_joint_4
-            name_joint_hand
-            joint_1_lower_limit
-            joint_1_upper_limit
-            joint_2_lower_limit
-            joint_2_upper_limit
-            joint_3_lower_limit
-            joint_3_upper_limit
-            joint_4_lower_limit
-            joint_4_upper_limit
-            joint_hand_lower_limit
-            joint_hand_upper_limit
-            port_name
-            baudrate
-            timeout_seconds
-            read_velocities
-            read_loads
-            read_voltages
-            read_temperatures
-            use_mock_components">
-    <ros2_control name="${name}" type="system">
+  <xacro:macro name="crane_plus_ros2_control_settings">
+    <ros2_control name="crane_plus" type="system">
       <hardware>
-        <xacro:if value="${use_mock_components}">
+        <xacro:if value="${USE_MOCK_COMPONENTS}">
           <plugin>mock_components/GenericSystem</plugin>
         </xacro:if>
-        <xacro:unless value="${use_mock_components}">
+        <xacro:unless value="${USE_MOCK_COMPONENTS}">
           <plugin>crane_plus_hardware/CranePlusHardware</plugin>
-          <param name="port_name">${port_name}</param>
-          <param name="baudrate">${baudrate}</param>
-          <param name="timeout_seconds">${timeout_seconds}</param>
-          <param name="read_velocities">${read_velocities}</param>
-          <param name="read_loads">${read_loads}</param>
-          <param name="read_voltages">${read_voltages}</param>
-          <param name="read_temperatures">${read_temperatures}</param>
+          <param name="port_name">${PORT_NAME}</param>
+          <param name="baudrate">${BAUDRATE}</param>
+          <param name="timeout_seconds">${TIMEOUT_SECONDS}</param>
+          <param name="read_velocities">${READ_VELOCITIES}</param>
+          <param name="read_loads">${READ_LOADS}</param>
+          <param name="read_voltages">${READ_VOLTAGES}</param>
+          <param name="read_temperatures">${READ_TEMPERATURES}</param>
         </xacro:unless>
       </hardware>
-      <joint name="${name_joint_1}">
+      <joint name="${NAME_JOINT_1}">
         <command_interface name="position">
-          <param name="min">${joint_1_lower_limit}</param>
-          <param name="max">${joint_1_upper_limit}</param>
+          <param name="min">${JOINT_1_LOWER_LIMIT}</param>
+          <param name="max">${JOINT_1_UPPER_LIMIT}</param>
         </command_interface>
         <state_interface name="position"/>
@@ -54,8 +30,8 @@
         <param name="dxl_id">1</param>
       </joint>
-      <joint name="${name_joint_2}">
+      <joint name="${NAME_JOINT_2}">
         <command_interface name="position">
-          <param name="min">${joint_2_lower_limit}</param>
-          <param name="max">${joint_2_upper_limit}</param>
+          <param name="min">${JOINT_2_LOWER_LIMIT}</param>
+          <param name="max">${JOINT_2_UPPER_LIMIT}</param>
         </command_interface>
         <state_interface name="position"/>
@@ -66,8 +42,8 @@
         <param name="dxl_id">2</param>
       </joint>
-      <joint name="${name_joint_3}">
+      <joint name="${NAME_JOINT_3}">
         <command_interface name="position">
-          <param name="min">${joint_3_lower_limit}</param>
-          <param name="max">${joint_3_upper_limit}</param>
+          <param name="min">${JOINT_3_LOWER_LIMIT}</param>
+          <param name="max">${JOINT_3_UPPER_LIMIT}</param>
         </command_interface>
         <state_interface name="position"/>
@@ -78,8 +54,8 @@
         <param name="dxl_id">3</param>
       </joint>
-      <joint name="${name_joint_4}">
+      <joint name="${NAME_JOINT_4}">
         <command_interface name="position">
-          <param name="min">${joint_4_lower_limit}</param>
-          <param name="max">${joint_4_upper_limit}</param>
+          <param name="min">${JOINT_4_LOWER_LIMIT}</param>
+          <param name="max">${JOINT_4_UPPER_LIMIT}</param>
         </command_interface>
         <state_interface name="position"/>
@@ -90,8 +66,8 @@
         <param name="dxl_id">4</param>
       </joint>
-      <joint name="${name_joint_hand}">
+      <joint name="${NAME_JOINT_HAND}">
         <command_interface name="position">
-          <param name="min">${joint_hand_lower_limit}</param>
-          <param name="max">${joint_hand_upper_limit}</param>
+          <param name="min">${JOINT_HAND_LOWER_LIMIT}</param>
+          <param name="max">${JOINT_HAND_UPPER_LIMIT}</param>
         </command_interface>
         <state_interface name="position"/>

File: crane_plus_description/urdf/crane_plus.urdf.xacro (robot description, xacro)
@@ -18,4 +18,12 @@
   <xacro:arg name="gz_control_config_file_path" default="" />
   <xacro:property name="USE_CAMERA" value="$(arg use_camera)"/>
+  <xacro:property name="USE_MOCK_COMPONENTS" value="$(arg use_mock_components)"/>
+  <xacro:property name="PORT_NAME" value="$(arg port_name)"/>
+  <xacro:property name="BAUDRATE" value="$(arg baudrate)"/>
+  <xacro:property name="TIMEOUT_SECONDS" value="$(arg timeout_seconds)"/>
+  <xacro:property name="READ_VELOCITIES" value="$(arg read_velocities)"/>
+  <xacro:property name="READ_LOADS" value="$(arg read_loads)"/>
+  <xacro:property name="READ_VOLTAGES" value="$(arg read_voltages)"/>
+  <xacro:property name="READ_TEMPERATURES" value="$(arg read_temperatures)"/>
   <xacro:property name="GZ_CONTROL_CONFIG_PACKAGE" value="$(arg gz_control_config_package)"/>
   <xacro:property name="GZ_CONTROL_CONFIG_FILE_PATH" value="$(arg gz_control_config_file_path)"/>
@@ -57,29 +65,5 @@
   </xacro:crane_plus>
   <xacro:unless value="$(arg use_gazebo)">
-    <xacro:crane_plus_ros2_control_settings
-      name="crane_plus"
-      name_joint_1="${NAME_JOINT_1}"
-      name_joint_2="${NAME_JOINT_2}"
-      name_joint_3="${NAME_JOINT_3}"
-      name_joint_4="${NAME_JOINT_4}"
-      name_joint_hand="${NAME_JOINT_HAND}"
-      joint_1_lower_limit="${JOINT_1_LOWER_LIMIT}"
-      joint_1_upper_limit="${JOINT_1_UPPER_LIMIT}"
-      joint_2_lower_limit="${JOINT_2_LOWER_LIMIT}"
-      joint_2_upper_limit="${JOINT_2_UPPER_LIMIT}"
-      joint_3_lower_limit="${JOINT_3_LOWER_LIMIT}"
-      joint_3_upper_limit="${JOINT_3_UPPER_LIMIT}"
-      joint_4_lower_limit="${JOINT_4_LOWER_LIMIT}"
-      joint_4_upper_limit="${JOINT_4_UPPER_LIMIT}"
-      joint_hand_lower_limit="${JOINT_HAND_LOWER_LIMIT}"
-      joint_hand_upper_limit="${JOINT_HAND_UPPER_LIMIT}"
-      port_name="$(arg port_name)"
-      baudrate="$(arg baudrate)"
-      timeout_seconds="$(arg timeout_seconds)"
-      read_velocities="$(arg read_velocities)"
-      read_loads="$(arg read_loads)"
-      read_voltages="$(arg read_voltages)"
-      read_temperatures="$(arg read_temperatures)"
-      use_mock_components="$(arg use_mock_components)" />
+    <xacro:crane_plus_ros2_control_settings />
   </xacro:unless>
   <xacro:if value="$(arg use_gazebo)">
