Commit message: カメラスタンドのリンク名を変更、マテリアルを定義して使い回す

File: crane_plus_description/urdf/camera_stand.urdf.xacro (robot description, xacro)
@@ -1,6 +1,9 @@
 <?xml version="1.0"?>
-<robot name="camera_stand_parts" xmlns:xacro="http://www.ros.org/wiki/xacro">
+<robot name="camera_stand" xmlns:xacro="http://www.ros.org/wiki/xacro">
+  <material name="grey">
+    <color rgba="0.8 0.8 0.8 1.0" />
+  </material>
   <xacro:macro name="camera_stand" params="parent">
-    <link name="camera_stand_p1">
+    <link name="camera_stand_link1">
       <visual>
         <origin xyz="0 0 0" rpy="0 0 0" />
@@ -8,7 +11,5 @@
           <box size="0.02 0.285 0.02" />
         </geometry>
-        <material name="grey">
-          <color rgba="0.8 0.8 0.8 1.0" />
-        </material>
+        <material name="grey" />
       </visual>
       <collision>
@@ -17,4 +18,5 @@
           <box size="0.02 0.285 0.02" />
         </geometry>
+        <material name="grey" />
       </collision>
     </link>
@@ -22,7 +24,7 @@
       <origin xyz="-0.052 0.08 0.01" rpy="0 0 0" />
       <parent link="${parent}" />
-      <child link="camera_stand_p1" />
+      <child link="camera_stand_link1" />
     </joint>
-    <link name="camera_stand_p2">
+    <link name="camera_stand_link2">
       <visual>
         <origin xyz="0 0 0" rpy="0 0 0" />
@@ -30,7 +32,5 @@
           <box size="0.02 0.02 0.44" />
         </geometry>
-        <material name="grey">
-          <color rgba="0.8 0.8 0.8 1.0" />
-        </material>
+        <material name="grey" />
       </visual>
       <collision>
@@ -39,12 +39,13 @@
           <box size="0.02 0.02 0.44" />
         </geometry>
+        <material name="grey" />
       </collision>
     </link>
     <joint name="camera_stand_joint2" type="fixed">
       <origin xyz="0 0.02253 0.23" rpy="0 0 0" />
-      <parent link="camera_stand_p1" />
-      <child link="camera_stand_p2" />
+      <parent link="camera_stand_link1" />
+      <child link="camera_stand_link2" />
     </joint>
-    <link name="camera_stand_p3">
+    <link name="camera_stand_link3">
       <visual>
         <origin xyz="0 0 0" rpy="0 0 0" />
@@ -52,7 +53,5 @@
           <box size="0.13 0.02 0.02" />
         </geometry>
-        <material name="grey">
-          <color rgba="0.8 0.8 0.8 1.0" />
-        </material>
+        <material name="grey" />
       </visual>
       <collision>
@@ -61,12 +60,13 @@
           <box size="0.129 0.02 0.02" />
         </geometry>
+        <material name="grey" />
       </collision>
     </link>
     <joint name="camera_stand_joint3" type="fixed">
       <origin xyz="0.075 0 0.21" rpy="0 0 0" />
-      <parent link="camera_stand_p2" />
-      <child link="camera_stand_p3" />
+      <parent link="camera_stand_link2" />
+      <child link="camera_stand_link3" />
     </joint>
-    <link name="camera_stand_p4">
+    <link name="camera_stand_link4">
       <visual>
         <origin xyz="0 0 0" rpy="0 0 0" />
@@ -74,7 +74,5 @@
           <box size="0.055 0.02 0.02" />
         </geometry>
-        <material name="grey">
-          <color rgba="0.8 0.8 0.8 1.0" />
-        </material>
+        <material name="grey" />
       </visual>
       <collision>
@@ -83,12 +81,13 @@
           <box size="0.054 0.019 0.02" />
         </geometry>
+        <material name="grey" />
       </collision>
     </link>
     <joint name="camera_stand_joint4" type="fixed">
       <origin xyz="0.0375 -0.1325 0" rpy="0 0 0" />
-      <parent link="camera_stand_p1" />
-      <child link="camera_stand_p4" />
+      <parent link="camera_stand_link1" />
+      <child link="camera_stand_link4" />
     </joint>
-    <link name="camera_stand_p5">
+    <link name="camera_stand_link5">
       <visual>
         <origin xyz="0 0 0" rpy="0 0 0" />
@@ -96,7 +95,5 @@
           <box size="0.055 0.02 0.02" />
         </geometry>
-        <material name="grey">
-          <color rgba="0.8 0.8 0.8 1.0" />
-        </material>
+        <material name="grey" />
       </visual>
       <collision>
@@ -105,10 +102,11 @@
           <box size="0.054 0.02 0.02" />
         </geometry>
+        <material name="grey" />
       </collision>
     </link>
     <joint name="camera_stand_joint5" type="fixed">
       <origin xyz="0.0375 0.1325 0" rpy="0 0 0" />
-      <parent link="camera_stand_p1" />
-      <child link="camera_stand_p5" />
+      <parent link="camera_stand_link1" />
+      <child link="camera_stand_link5" />
     </joint>
   </xacro:macro>
