Commit message: Fix joint limits

File: crane_plus_description/urdf/crane_plus.urdf.xacro (robot description, xacro)
@@ -15,16 +15,17 @@
   <!--   <child link="base_link"/>                          -->
   <!-- </joint>                                             -->
+  <xacro:property name="M_PI" value="3.14159"/>
   <crane_plus parent="base_link"
     joints_vlimit="2.0"
-    joint1_lower_limit="-1.57"
-    joint1_upper_limit="1.57"
-    joint2_lower_limit="-1.57"
-    joint2_upper_limit="1.57"
-    joint3_lower_limit="-1.57"
-    joint3_upper_limit="1.57"
-    joint4_lower_limit="-1.57"
-    joint4_upper_limit="1.57"
-    joint_hand_lower_limit="-1.57"
-    joint_hand_upper_limit="1.57">
+    joint1_lower_limit="-${M_PI*5/6}"
+    joint1_upper_limit="${M_PI*5/6}"
+    joint2_lower_limit="-${M_PI*0.5776}"
+    joint2_upper_limit="${M_PI*0.5612}"
+    joint3_lower_limit="-${M_PI*0.8105}"
+    joint3_upper_limit="${M_PI*0.7770}"
+    joint4_lower_limit="-${M_PI*0.5776}"
+    joint4_upper_limit="${M_PI*0.5564}"
+    joint_hand_lower_limit="-${M_PI*0.2191}"
+    joint_hand_upper_limit="${M_PI*0.2093}">
     <origin xyz="0 0 0"/>
   </crane_plus>

File: crane_plus_description/urdf/crane_plus.xacro (robot description, xacro)
@@ -19,5 +19,4 @@
     <color rgba="0.3 0.3 1.0 1.0"/>
   </material>
-  <xacro:property name="M_PI" value="3.14159"/>
   <xacro:property name="SCALE_MM" value="0.001"/>
   <xacro:property name="SCALE_CM" value="0.01"/>

Commit message: Add crane_plus_gazebo. Spawn CRANE+ and table and box

File: crane_plus_description/urdf/crane_plus.urdf.xacro (robot description, xacro)
@@ -8,13 +8,13 @@
   <xacro:include filename="$(find crane_plus_description)/urdf/crane_plus.xacro"/>
   <!-- Link to provide the location reference for the arm -->
-  <!-- <link name="base_link"/> -->
+  <link name="base_link"/>
   <!-- Used for fixing robot to Gazebo 'base_link' -->
-  <!-- <link name="world"/>                                 -->
-  <!-- <joint name="base_link_to_world_joint" type="fixed"> -->
-  <!--   <parent link="world"/>                             -->
-  <!--   <child link="base_link"/>                          -->
-  <!-- </joint>                                             -->
+  <link name="world"/>
+  <joint name="base_link_to_world_joint" type="fixed">
+    <parent link="world"/>
+    <child link="base_link"/>
+  </joint>
   <xacro:property name="M_PI" value="3.14159"/>
-  <crane_plus parent="base_link"
+  <xacro:crane_plus parent="base_link"
     joints_vlimit="2.0"
     joint1_lower_limit="-${M_PI*5/6}"
@@ -29,4 +29,4 @@
     joint_hand_upper_limit="${M_PI*0.2093}">
     <origin xyz="0 0 0"/>
-  </crane_plus>
+  </xacro:crane_plus>
 </robot>

File: crane_plus_description/urdf/crane_plus.xacro (robot description, xacro)
@@ -27,5 +27,5 @@
   <xacro:property name="NAME_JOINT_4" value="crane_plus_joint4"/>
   <xacro:property name="NAME_JOINT_HAND" value="crane_plus_joint_hand"/>
-  <xacro:property name="NAME_LINK_BASE" value="base_link"/>
+  <xacro:property name="NAME_LINK_BASE" value="crane_plus_base"/>
   <xacro:property name="NAME_LINK_1" value="crane_plus_link1"/>
   <xacro:property name="NAME_LINK_2" value="crane_plus_link2"/>
@@ -47,9 +47,9 @@
               joint_hand_upper_limit
               *origin">
-    <!-- <joint name="${NAME_JOINT_BASE}" type="fixed"> -->
-    <!--   <xacro:insert_block name="origin"/>          -->
-    <!--   <parent link="${parent}"/>                   -->
-    <!--   <child link="${NAME_LINK_BASE}"/>            -->
-    <!-- </joint>                                       -->
+    <joint name="${NAME_JOINT_BASE}" type="fixed">
+      <xacro:insert_block name="origin"/>
+      <parent link="${parent}"/>
+      <child link="${NAME_LINK_BASE}"/>
+    </joint>
     <link name="${NAME_LINK_BASE}">
       <visual>
@@ -67,4 +67,8 @@
         </geometry>
       </collision>
+      <inertial>
+        <mass value="1"/>
+        <inertia ixx="1" ixy="0.0" ixz="0.0" iyy="1" iyz="0.0" izz="1"/>
+      </inertial>
     </link>
     <joint name="${NAME_JOINT_1}" type="revolute">
@@ -96,4 +100,8 @@
         </geometry>
       </collision>
+      <inertial>
+        <mass value="1"/>
+        <inertia ixx="1" ixy="0.0" ixz="0.0" iyy="1" iyz="0.0" izz="1"/>
+      </inertial>
     </link>
     <joint name="${NAME_JOINT_2}" type="revolute">
@@ -125,4 +133,8 @@
         </geometry>
       </collision>
+      <inertial>
+        <mass value="1"/>
+        <inertia ixx="1" ixy="0.0" ixz="0.0" iyy="1" iyz="0.0" izz="1"/>
+      </inertial>
     </link>
     <joint name="${NAME_JOINT_3}" type="revolute">
@@ -154,4 +166,8 @@
         </geometry>
       </collision>
+      <inertial>
+        <mass value="1"/>
+        <inertia ixx="1" ixy="0.0" ixz="0.0" iyy="1" iyz="0.0" izz="1"/>
+      </inertial>
     </link>
     <joint name="${NAME_JOINT_4}" type="revolute">
@@ -183,4 +199,8 @@
         </geometry>
       </collision>
+      <inertial>
+        <mass value="1"/>
+        <inertia ixx="1" ixy="0.0" ixz="0.0" iyy="1" iyz="0.0" izz="1"/>
+      </inertial>
     </link>
     <joint name="${NAME_JOINT_HAND}" type="revolute">
@@ -212,4 +232,8 @@
         </geometry>
       </collision>
+      <inertial>
+        <mass value="1"/>
+        <inertia ixx="1" ixy="0.0" ixz="0.0" iyy="1" iyz="0.0" izz="1"/>
+      </inertial>
     </link>
   </xacro:macro>

Commit message: Update joint_limits of xacro file

File: crane_plus_description/urdf/crane_plus.urdf.xacro (robot description, xacro)
@@ -16,16 +16,18 @@
   </joint>
   <xacro:property name="M_PI" value="3.14159"/>
+  <xacro:property name="TO_RADIAN" value="${M_PI / 180.0}"/>
+  <xacro:property name="SERVO_HOME" value="${TO_RADIAN * 150.0}"/>
   <xacro:crane_plus parent="base_link"
     joints_vlimit="2.0"
-    joint1_lower_limit="-${M_PI*5/6}"
-    joint1_upper_limit="${M_PI*5/6}"
-    joint2_lower_limit="-${M_PI*0.5776}"
-    joint2_upper_limit="${M_PI*0.5612}"
-    joint3_lower_limit="-${M_PI*0.8105}"
-    joint3_upper_limit="${M_PI*0.7770}"
-    joint4_lower_limit="-${M_PI*0.5776}"
-    joint4_upper_limit="${M_PI*0.5564}"
-    joint_hand_lower_limit="-${M_PI*0.2191}"
-    joint_hand_upper_limit="${M_PI*0.2093}">
+    joint1_lower_limit="${0.0 * TO_RADIAN - SERVO_HOME}"
+    joint1_upper_limit="${300.0 * TO_RADIAN - SERVO_HOME}"
+    joint2_lower_limit="${45.45 * TO_RADIAN - SERVO_HOME}"
+    joint2_upper_limit="${252.20 * TO_RADIAN - SERVO_HOME}"
+    joint3_lower_limit="${3.52 * TO_RADIAN - SERVO_HOME}"
+    joint3_upper_limit="${290.62 * TO_RADIAN - SERVO_HOME}"
+    joint4_lower_limit="${44.57 * TO_RADIAN - SERVO_HOME}"
+    joint4_upper_limit="${251.32 * TO_RADIAN - SERVO_HOME}"
+    joint_hand_lower_limit="${109.38 * TO_RADIAN - SERVO_HOME}"
+    joint_hand_upper_limit="${188.27 * TO_RADIAN - SERVO_HOME}">
     <origin xyz="0 0 0"/>
   </xacro:crane_plus>

Commit message: Spawn two CRANE+V2 models (one is not stable).

File: crane_plus_description/urdf/crane_plus.urdf.xacro (robot description, xacro)
@@ -18,5 +18,7 @@
   <xacro:property name="TO_RADIAN" value="${M_PI / 180.0}"/>
   <xacro:property name="SERVO_HOME" value="${TO_RADIAN * 150.0}"/>
-  <xacro:crane_plus parent="base_link"
+  <xacro:crane_plus
+    prefix="right_crane_plus"
+    parent="base_link"
     joints_vlimit="2.0"
     joint1_lower_limit="${0.0 * TO_RADIAN - SERVO_HOME}"
@@ -30,5 +32,27 @@
     joint_hand_lower_limit="${109.38 * TO_RADIAN - SERVO_HOME}"
     joint_hand_upper_limit="${188.27 * TO_RADIAN - SERVO_HOME}">
-    <origin xyz="0 0 0"/>
+    <origin xyz="0 -0.2 0.0"/>
   </xacro:crane_plus>
+  <xacro:crane_plus
+    prefix="left_crane_plus"
+    parent="base_link"
+    joints_vlimit="2.0"
+    joint1_lower_limit="${0.0 * TO_RADIAN - SERVO_HOME}"
+    joint1_upper_limit="${300.0 * TO_RADIAN - SERVO_HOME}"
+    joint2_lower_limit="${45.45 * TO_RADIAN - SERVO_HOME}"
+    joint2_upper_limit="${252.20 * TO_RADIAN - SERVO_HOME}"
+    joint3_lower_limit="${3.52 * TO_RADIAN - SERVO_HOME}"
+    joint3_upper_limit="${290.62 * TO_RADIAN - SERVO_HOME}"
+    joint4_lower_limit="${44.57 * TO_RADIAN - SERVO_HOME}"
+    joint4_upper_limit="${251.32 * TO_RADIAN - SERVO_HOME}"
+    joint_hand_lower_limit="${109.38 * TO_RADIAN - SERVO_HOME}"
+    joint_hand_upper_limit="${188.27 * TO_RADIAN - SERVO_HOME}">
+    <origin xyz="0 0.2 0"/>
+  </xacro:crane_plus>
+  <gazebo>
+    <plugin filename="libgazebo_ros2_control.so" name="gazebo_ros2_control">
+      <robot_sim_type>gazebo_ros2_control/GazeboSystem</robot_sim_type>
+      <parameters>$(find crane_plus_gazebo)/config/gazebo_controllers.yaml</parameters>
+    </plugin>
+  </gazebo>
 </robot>

File: crane_plus_description/urdf/crane_plus.xacro (robot description, xacro)
@@ -24,16 +24,4 @@
   <xacro:property name="SCALE_MM" value="0.001"/>
   <xacro:property name="SCALE_CM" value="0.01"/>
-  <xacro:property name="NAME_JOINT_BASE" value="crane_plus_joint_base"/>
-  <xacro:property name="NAME_JOINT_1" value="crane_plus_joint1"/>
-  <xacro:property name="NAME_JOINT_2" value="crane_plus_joint2"/>
-  <xacro:property name="NAME_JOINT_3" value="crane_plus_joint3"/>
-  <xacro:property name="NAME_JOINT_4" value="crane_plus_joint4"/>
-  <xacro:property name="NAME_JOINT_HAND" value="crane_plus_joint_hand"/>
-  <xacro:property name="NAME_LINK_BASE" value="crane_plus_base"/>
-  <xacro:property name="NAME_LINK_1" value="crane_plus_link1"/>
-  <xacro:property name="NAME_LINK_2" value="crane_plus_link2"/>
-  <xacro:property name="NAME_LINK_3" value="crane_plus_link3"/>
-  <xacro:property name="NAME_LINK_4" value="crane_plus_link4"/>
-  <xacro:property name="NAME_LINK_HAND" value="crane_plus_link_hand"/>
   <xacro:property name="MESH_LINK_BASE" value="crane_plus_description/meshes/visual/body_20201013.stl"/>
   <xacro:property name="MESH_LINK_1" value="crane_plus_description/meshes/visual/Link1_20201013.stl"/>
@@ -49,5 +37,6 @@
   <xacro:property name="MESH_COLLISION_LINK_HAND" value="crane_plus_description/meshes/collision/Hand_collision_20201013.stl"/>
   <xacro:macro name="crane_plus"
-      params="parent
+      params="prefix
+              parent
               joints_vlimit
               joint1_lower_limit
@@ -62,4 +51,16 @@
               joint_hand_upper_limit
               *origin">
+    <xacro:property name="NAME_JOINT_BASE" value="${prefix}_joint_base"/>
+    <xacro:property name="NAME_JOINT_1" value="${prefix}_joint1"/>
+    <xacro:property name="NAME_JOINT_2" value="${prefix}_joint2"/>
+    <xacro:property name="NAME_JOINT_3" value="${prefix}_joint3"/>
+    <xacro:property name="NAME_JOINT_4" value="${prefix}_joint4"/>
+    <xacro:property name="NAME_JOINT_HAND" value="${prefix}_joint_hand"/>
+    <xacro:property name="NAME_LINK_BASE" value="${prefix}_base"/>
+    <xacro:property name="NAME_LINK_1" value="${prefix}_link1"/>
+    <xacro:property name="NAME_LINK_2" value="${prefix}_link2"/>
+    <xacro:property name="NAME_LINK_3" value="${prefix}_link3"/>
+    <xacro:property name="NAME_LINK_4" value="${prefix}_link4"/>
+    <xacro:property name="NAME_LINK_HAND" value="${prefix}_link_hand"/>
     <joint name="${NAME_JOINT_BASE}" type="fixed">
       <xacro:insert_block name="origin"/>
@@ -288,5 +289,5 @@
       joint_hand_upper_limit="${joint_hand_upper_limit}" /> -->
     <xacro:crane_plus_gazebo_ros2_control_settings
-      name="GazeboSystem"
+      name="${prefix}_GazeboSystem"
       name_joint_1="${NAME_JOINT_1}"
       name_joint_2="${NAME_JOINT_2}"
