Commit message: Load ros2_control.xacro from crane_plus.xacro. This makes using gazebo_ros2_control easier.

File: crane_plus_description/urdf/crane_plus.urdf.xacro (robot description, xacro)
@@ -7,4 +7,5 @@
     xmlns:interface="http://playerstage.sourceforge.net/gazebo/xmlschema/#interface">
   <xacro:include filename="$(find crane_plus_description)/urdf/crane_plus.xacro"/>
+  <xacro:include filename="$(find crane_plus_description)/urdf/crane_plus.ros2_control.xacro"/>
   <!-- Link to provide the location reference for the arm -->
   <link name="base_link"/>
@@ -15,20 +16,73 @@
     <child link="base_link"/>
   </joint>
+  <xacro:property name="NAME_LINK_BASE" value="crane_plus_base"/>
+  <xacro:property name="NAME_LINK_1" value="crane_plus_link1"/>
+  <xacro:property name="NAME_LINK_2" value="crane_plus_link2"/>
+  <xacro:property name="NAME_LINK_3" value="crane_plus_link3"/>
+  <xacro:property name="NAME_LINK_4" value="crane_plus_link4"/>
+  <xacro:property name="NAME_LINK_HAND" value="crane_plus_link_hand"/>
+  <xacro:property name="NAME_JOINT_BASE" value="crane_plus_joint_base"/>
+  <xacro:property name="NAME_JOINT_1" value="crane_plus_joint1"/>
+  <xacro:property name="NAME_JOINT_2" value="crane_plus_joint2"/>
+  <xacro:property name="NAME_JOINT_3" value="crane_plus_joint3"/>
+  <xacro:property name="NAME_JOINT_4" value="crane_plus_joint4"/>
+  <xacro:property name="NAME_JOINT_HAND" value="crane_plus_joint_hand"/>
   <xacro:property name="M_PI" value="3.14159"/>
   <xacro:property name="TO_RADIAN" value="${M_PI / 180.0}"/>
   <xacro:property name="SERVO_HOME" value="${TO_RADIAN * 150.0}"/>
-  <xacro:crane_plus parent="base_link"
-    joints_vlimit="2.0"
-    joint1_lower_limit="${0.0 * TO_RADIAN - SERVO_HOME}"
-    joint1_upper_limit="${300.0 * TO_RADIAN - SERVO_HOME}"
-    joint2_lower_limit="${45.45 * TO_RADIAN - SERVO_HOME}"
-    joint2_upper_limit="${252.20 * TO_RADIAN - SERVO_HOME}"
-    joint3_lower_limit="${3.52 * TO_RADIAN - SERVO_HOME}"
-    joint3_upper_limit="${290.62 * TO_RADIAN - SERVO_HOME}"
-    joint4_lower_limit="${44.57 * TO_RADIAN - SERVO_HOME}"
-    joint4_upper_limit="${251.32 * TO_RADIAN - SERVO_HOME}"
-    joint_hand_lower_limit="${109.38 * TO_RADIAN - SERVO_HOME}"
-    joint_hand_upper_limit="${188.27 * TO_RADIAN - SERVO_HOME}">
+  <xacro:property name="JOINT_VELOCITY_LIMIT" value="2.0"/>
+  <xacro:property name="JOINT_1_LOWER_LIMIT" value="${0.0 * TO_RADIAN - SERVO_HOME}"/>
+  <xacro:property name="JOINT_1_UPPER_LIMIT" value="${300.0 * TO_RADIAN - SERVO_HOME}"/>
+  <xacro:property name="JOINT_2_LOWER_LIMIT" value="${45.45 * TO_RADIAN - SERVO_HOME}"/>
+  <xacro:property name="JOINT_2_UPPER_LIMIT" value="${252.20 * TO_RADIAN - SERVO_HOME}"/>
+  <xacro:property name="JOINT_3_LOWER_LIMIT" value="${3.52 * TO_RADIAN - SERVO_HOME}"/>
+  <xacro:property name="JOINT_3_UPPER_LIMIT" value="${290.62 * TO_RADIAN - SERVO_HOME}"/>
+  <xacro:property name="JOINT_4_LOWER_LIMIT" value="${44.57 * TO_RADIAN - SERVO_HOME}"/>
+  <xacro:property name="JOINT_4_UPPER_LIMIT" value="${251.32 * TO_RADIAN - SERVO_HOME}"/>
+  <xacro:property name="JOINT_HAND_LOWER_LIMIT" value="${109.38 * TO_RADIAN - SERVO_HOME}"/>
+  <xacro:property name="JOINT_HAND_UPPER_LIMIT" value="${188.27 * TO_RADIAN - SERVO_HOME}"/>
+  <xacro:crane_plus
+    parent="base_link"
+    name_link_base="${NAME_LINK_BASE}"
+    name_link_1="${NAME_LINK_1}"
+    name_link_2="${NAME_LINK_2}"
+    name_link_3="${NAME_LINK_3}"
+    name_link_4="${NAME_LINK_4}"
+    name_link_hand="${NAME_LINK_HAND}"
+    name_joint_base="${NAME_JOINT_BASE}"
+    name_joint_1="${NAME_JOINT_1}"
+    name_joint_2="${NAME_JOINT_2}"
+    name_joint_3="${NAME_JOINT_3}"
+    name_joint_4="${NAME_JOINT_4}"
+    name_joint_hand="${NAME_JOINT_HAND}"
+    joints_vlimit="${JOINT_VELOCITY_LIMIT}"
+    joint_1_lower_limit="${JOINT_1_LOWER_LIMIT}"
+    joint_1_upper_limit="${JOINT_1_UPPER_LIMIT}"
+    joint_2_lower_limit="${JOINT_2_LOWER_LIMIT}"
+    joint_2_upper_limit="${JOINT_2_UPPER_LIMIT}"
+    joint_3_lower_limit="${JOINT_3_LOWER_LIMIT}"
+    joint_3_upper_limit="${JOINT_3_UPPER_LIMIT}"
+    joint_4_lower_limit="${JOINT_4_LOWER_LIMIT}"
+    joint_4_upper_limit="${JOINT_4_UPPER_LIMIT}"
+    joint_hand_lower_limit="${JOINT_HAND_LOWER_LIMIT}"
+    joint_hand_upper_limit="${JOINT_HAND_UPPER_LIMIT}" >
     <origin xyz="0 0 0"/>
   </xacro:crane_plus>
+  <xacro:crane_plus_ros2_control_settings
+    name="crane_plus"
+    name_joint_1="${NAME_JOINT_1}"
+    name_joint_2="${NAME_JOINT_2}"
+    name_joint_3="${NAME_JOINT_3}"
+    name_joint_4="${NAME_JOINT_4}"
+    name_joint_hand="${NAME_JOINT_HAND}"
+    joint_1_lower_limit="${JOINT_1_LOWER_LIMIT}"
+    joint_1_upper_limit="${JOINT_1_UPPER_LIMIT}"
+    joint_2_lower_limit="${JOINT_2_LOWER_LIMIT}"
+    joint_2_upper_limit="${JOINT_2_UPPER_LIMIT}"
+    joint_3_lower_limit="${JOINT_3_LOWER_LIMIT}"
+    joint_3_upper_limit="${JOINT_3_UPPER_LIMIT}"
+    joint_4_lower_limit="${JOINT_4_LOWER_LIMIT}"
+    joint_4_upper_limit="${JOINT_4_UPPER_LIMIT}"
+    joint_hand_lower_limit="${JOINT_HAND_LOWER_LIMIT}"
+    joint_hand_upper_limit="${JOINT_HAND_UPPER_LIMIT}" />
 </robot>

File: crane_plus_description/urdf/crane_plus.xacro (robot description, xacro)
@@ -1,5 +1,4 @@
 <?xml version="1.0"?>
 <robot xmlns:xacro="http://ros.org/wiki/xacro">
-  <xacro:include filename="$(find crane_plus_description)/urdf/crane_plus.ros2_control.xacro"/>
   <material name="black">
     <color rgba="0.2 0.2 0.2 1.0"/>
@@ -22,16 +21,4 @@
   <xacro:property name="SCALE_MM" value="0.001"/>
   <xacro:property name="SCALE_CM" value="0.01"/>
-  <xacro:property name="NAME_JOINT_BASE" value="crane_plus_joint_base"/>
-  <xacro:property name="NAME_JOINT_1" value="crane_plus_joint1"/>
-  <xacro:property name="NAME_JOINT_2" value="crane_plus_joint2"/>
-  <xacro:property name="NAME_JOINT_3" value="crane_plus_joint3"/>
-  <xacro:property name="NAME_JOINT_4" value="crane_plus_joint4"/>
-  <xacro:property name="NAME_JOINT_HAND" value="crane_plus_joint_hand"/>
-  <xacro:property name="NAME_LINK_BASE" value="crane_plus_base"/>
-  <xacro:property name="NAME_LINK_1" value="crane_plus_link1"/>
-  <xacro:property name="NAME_LINK_2" value="crane_plus_link2"/>
-  <xacro:property name="NAME_LINK_3" value="crane_plus_link3"/>
-  <xacro:property name="NAME_LINK_4" value="crane_plus_link4"/>
-  <xacro:property name="NAME_LINK_HAND" value="crane_plus_link_hand"/>
   <xacro:property name="MESH_LINK_BASE" value="crane_plus_description/meshes/visual/body_20201013.stl"/>
   <xacro:property name="MESH_LINK_1" value="crane_plus_description/meshes/visual/Link1_20201013.stl"/>
@@ -48,22 +35,34 @@
   <xacro:macro name="crane_plus"
       params="parent
+              name_link_base
+              name_link_1
+              name_link_2
+              name_link_3
+              name_link_4
+              name_link_hand
+              name_joint_base
+              name_joint_1
+              name_joint_2
+              name_joint_3
+              name_joint_4
+              name_joint_hand
               joints_vlimit
-              joint1_lower_limit
-              joint1_upper_limit
-              joint2_lower_limit
-              joint2_upper_limit
-              joint3_lower_limit
-              joint3_upper_limit
-              joint4_lower_limit
-              joint4_upper_limit
+              joint_1_lower_limit
+              joint_1_upper_limit
+              joint_2_lower_limit
+              joint_2_upper_limit
+              joint_3_lower_limit
+              joint_3_upper_limit
+              joint_4_lower_limit
+              joint_4_upper_limit
               joint_hand_lower_limit
               joint_hand_upper_limit
               *origin">
-    <joint name="${NAME_JOINT_BASE}" type="fixed">
+    <joint name="${name_joint_base}" type="fixed">
       <xacro:insert_block name="origin"/>
       <parent link="${parent}"/>
-      <child link="${NAME_LINK_BASE}"/>
-    </joint>
-    <link name="${NAME_LINK_BASE}">
+      <child link="${name_link_base}"/>
+    </joint>
+    <link name="${name_link_base}">
       <visual>
         <origin xyz="0 0 0" rpy="0 0 0"/>
@@ -88,5 +87,5 @@
       </inertial>
     </link>
-    <joint name="${NAME_JOINT_1}" type="revolute">
+    <joint name="${name_joint_1}" type="revolute">
       <origin xyz="0 0 0.0454" rpy="0 0 0"/>
       <axis xyz="0 0 1"/>
@@ -94,12 +93,12 @@
         effort="10.0"
         velocity="${joints_vlimit}"
-        lower="${joint1_lower_limit}"
-        upper="${joint1_upper_limit}"
-        />
-      <parent link="${NAME_LINK_BASE}"/>
-      <child link="${NAME_LINK_1}"/>
-      <dynamics damping="1.0e-6" friction="2.0e-1"/>
-    </joint>
-    <link name="${NAME_LINK_1}">
+        lower="${joint_1_lower_limit}"
+        upper="${joint_1_upper_limit}"
+        />
+      <parent link="${name_link_base}"/>
+      <child link="${name_link_1}"/>
+      <dynamics damping="1.0e-6" friction="2.0e-1"/>
+    </joint>
+    <link name="${name_link_1}">
       <visual>
         <origin xyz="0 0 0" rpy="0 0 ${M_PI}"/>
@@ -124,5 +123,5 @@
       </inertial>
     </link>
-    <joint name="${NAME_JOINT_2}" type="revolute">
+    <joint name="${name_joint_2}" type="revolute">
       <origin xyz="0 0 0.026" rpy="0 0 0"/>
       <axis xyz="0 1 0"/>
@@ -130,12 +129,12 @@
         effort="10.0"
         velocity="${joints_vlimit}"
-        lower="${joint2_lower_limit}"
-        upper="${joint2_upper_limit}"
-        />
-      <parent link="${NAME_LINK_1}"/>
-      <child link="${NAME_LINK_2}"/>
-      <dynamics damping="1.0e-6" friction="2.0e-1"/>
-    </joint>
-    <link name="${NAME_LINK_2}">
+        lower="${joint_2_lower_limit}"
+        upper="${joint_2_upper_limit}"
+        />
+      <parent link="${name_link_1}"/>
+      <child link="${name_link_2}"/>
+      <dynamics damping="1.0e-6" friction="2.0e-1"/>
+    </joint>
+    <link name="${name_link_2}">
       <visual>
         <origin xyz="0 0 0" rpy="${M_PI/2} 0 0"/>
@@ -160,5 +159,5 @@
       </inertial>
     </link>
-    <joint name="${NAME_JOINT_3}" type="revolute">
+    <joint name="${name_joint_3}" type="revolute">
       <origin xyz="0 0 0.083" rpy="0 0 0"/>
       <axis xyz="0 -1 0"/>
@@ -166,12 +165,12 @@
         effort="10.0"
         velocity="${joints_vlimit}"
-        lower="${joint3_lower_limit}"
-        upper="${joint3_upper_limit}"
-        />
-      <parent link="${NAME_LINK_2}"/>
-      <child link="${NAME_LINK_3}"/>
-      <dynamics damping="1.0e-6" friction="2.0e-1"/>
-    </joint>
-    <link name="${NAME_LINK_3}">
+        lower="${joint_3_lower_limit}"
+        upper="${joint_3_upper_limit}"
+        />
+      <parent link="${name_link_2}"/>
+      <child link="${name_link_3}"/>
+      <dynamics damping="1.0e-6" friction="2.0e-1"/>
+    </joint>
+    <link name="${name_link_3}">
       <visual>
         <origin xyz="0 0 0" rpy="${M_PI/2} 0 0"/>
@@ -196,5 +195,5 @@
       </inertial>
     </link>
-    <joint name="${NAME_JOINT_4}" type="revolute">
+    <joint name="${name_joint_4}" type="revolute">
       <origin xyz="0 0 0.0935" rpy="0 0 0"/>
       <axis xyz="0 -1 0"/>
@@ -202,12 +201,12 @@
         effort="10.0"
         velocity="${joints_vlimit}"
-        lower="${joint4_lower_limit}"
-        upper="${joint4_upper_limit}"
-        />
-      <parent link="${NAME_LINK_3}"/>
-      <child link="${NAME_LINK_4}"/>
-      <dynamics damping="1.0e-6" friction="2.0e-1"/>
-    </joint>
-    <link name="${NAME_LINK_4}">
+        lower="${joint_4_lower_limit}"
+        upper="${joint_4_upper_limit}"
+        />
+      <parent link="${name_link_3}"/>
+      <child link="${name_link_4}"/>
+      <dynamics damping="1.0e-6" friction="2.0e-1"/>
+    </joint>
+    <link name="${name_link_4}">
       <visual>
         <origin xyz="0 0 0" rpy="${M_PI/2} 0 0"/>
@@ -232,5 +231,5 @@
       </inertial>
     </link>
-    <joint name="${NAME_JOINT_HAND}" type="revolute">
+    <joint name="${name_joint_hand}" type="revolute">
       <origin xyz="0 -0.0145 0.045" rpy="0 0 0"/>
       <axis xyz="-1 0 0"/>
@@ -241,9 +240,9 @@
         upper="${joint_hand_upper_limit}"
         />
-      <parent link="${NAME_LINK_4}"/>
-      <child link="${NAME_LINK_HAND}"/>
-      <dynamics damping="1.0e-6" friction="2.0e-1"/>
-    </joint>
-    <link name="${NAME_LINK_HAND}">
+      <parent link="${name_link_4}"/>
+      <child link="${name_link_hand}"/>
+      <dynamics damping="1.0e-6" friction="2.0e-1"/>
+    </joint>
+    <link name="${name_link_hand}">
       <visual>
         <origin xyz="0 0 0" rpy="0 -${M_PI/2} 0"/>
@@ -268,21 +267,4 @@
       </inertial>
     </link>
-    <xacro:crane_plus_ros2_control_settings
-      name="crane_plus"
-      name_joint_1="${NAME_JOINT_1}"
-      name_joint_2="${NAME_JOINT_2}"
-      name_joint_3="${NAME_JOINT_3}"
-      name_joint_4="${NAME_JOINT_4}"
-      name_joint_hand="${NAME_JOINT_HAND}"
-      joint_1_lower_limit="${joint1_lower_limit}"
-      joint_1_upper_limit="${joint1_upper_limit}"
-      joint_2_lower_limit="${joint2_lower_limit}"
-      joint_2_upper_limit="${joint2_upper_limit}"
-      joint_3_lower_limit="${joint3_lower_limit}"
-      joint_3_upper_limit="${joint3_upper_limit}"
-      joint_4_lower_limit="${joint4_lower_limit}"
-      joint_4_upper_limit="${joint4_upper_limit}"
-      joint_hand_lower_limit="${joint_hand_lower_limit}"
-      joint_hand_upper_limit="${joint_hand_upper_limit}" />
   </xacro:macro>
 </robot>

Commit message: MoveItの手先をjoint4からグリッパの中心へ変更

File: crane_plus_description/urdf/crane_plus.urdf.xacro (robot description, xacro)
@@ -36,4 +36,5 @@
   <xacro:property name="NAME_LINK_4" value="crane_plus_link4"/>
   <xacro:property name="NAME_LINK_HAND" value="crane_plus_link_hand"/>
+  <xacro:property name="NAME_LINK_ENDTIP" value="crane_plus_link_endtip"/>
   <xacro:property name="NAME_JOINT_BASE" value="crane_plus_joint_base"/>
   <xacro:property name="NAME_JOINT_1" value="crane_plus_joint1"/>
@@ -42,4 +43,5 @@
   <xacro:property name="NAME_JOINT_4" value="crane_plus_joint4"/>
   <xacro:property name="NAME_JOINT_HAND" value="crane_plus_joint_hand"/>
+  <xacro:property name="NAME_JOINT_ENDTIP" value="crane_plus_joint_endtip"/>
   <xacro:property name="M_PI" value="3.14159"/>
   <xacro:property name="TO_RADIAN" value="${M_PI / 180.0}"/>
@@ -64,4 +66,5 @@
     name_link_4="${NAME_LINK_4}"
     name_link_hand="${NAME_LINK_HAND}"
+    name_link_endtip="${NAME_LINK_ENDTIP}"
     name_joint_base="${NAME_JOINT_BASE}"
     name_joint_1="${NAME_JOINT_1}"
@@ -70,4 +73,5 @@
     name_joint_4="${NAME_JOINT_4}"
     name_joint_hand="${NAME_JOINT_HAND}"
+    name_joint_endtip="${NAME_JOINT_ENDTIP}"
     joints_vlimit="${JOINT_VELOCITY_LIMIT}"
     joint_1_lower_limit="${JOINT_1_LOWER_LIMIT}"

File: crane_plus_description/urdf/crane_plus.xacro (robot description, xacro)
@@ -41,4 +41,5 @@
               name_link_4
               name_link_hand
+              name_link_endtip
               name_joint_base
               name_joint_1
@@ -47,4 +48,5 @@
               name_joint_4
               name_joint_hand
+              name_joint_endtip
               joints_vlimit
               joint_1_lower_limit
@@ -268,4 +270,12 @@
       </inertial>
     </link>
+    <!-- endtip for MoveIt -->
+    <joint name="${name_joint_endtip}" type="fixed">
+      <origin xyz="0 0 0.090" rpy="0 ${-M_PI/2} 0"/>
+      <parent link="${name_link_4}"/>
+      <child link="${name_link_endtip}"/>
+    </joint>
+    <link name="${name_link_endtip}">
+    </link>
     <!-- camera -->
     <xacro:if value="$(arg use_camera)">

Commit message: Update crane_plus_description/urdf/crane_plus.urdf.xacro
Co-authored-by: Kuwamai <mitsumex333@gmail.com>

File: crane_plus_description/urdf/crane_plus.urdf.xacro (robot description, xacro)
@@ -36,5 +36,5 @@
   <xacro:property name="NAME_LINK_4" value="crane_plus_link4"/>
   <xacro:property name="NAME_LINK_HAND" value="crane_plus_link_hand"/>
-  <xacro:property name="NAME_LINK_ENDTIP" value="crane_plus_link_endtip"/>
+  <xacro:property name="NAME_LINK_TCP" value="crane_plus_link_tcp"/>
   <xacro:property name="NAME_JOINT_BASE" value="crane_plus_joint_base"/>
   <xacro:property name="NAME_JOINT_1" value="crane_plus_joint1"/>

Commit message: Update crane_plus_description/urdf/crane_plus.urdf.xacro
Co-authored-by: Kuwamai <mitsumex333@gmail.com>

File: crane_plus_description/urdf/crane_plus.urdf.xacro (robot description, xacro)
@@ -43,5 +43,5 @@
   <xacro:property name="NAME_JOINT_4" value="crane_plus_joint4"/>
   <xacro:property name="NAME_JOINT_HAND" value="crane_plus_joint_hand"/>
-  <xacro:property name="NAME_JOINT_ENDTIP" value="crane_plus_joint_endtip"/>
+  <xacro:property name="NAME_JOINT_TCP" value="crane_plus_joint_tcp"/>
   <xacro:property name="M_PI" value="3.14159"/>
   <xacro:property name="TO_RADIAN" value="${M_PI / 180.0}"/>

Commit message: arm_tcpを新設 - リンク名とジョイント名をendtipからtcpに変更（残っていた分） - arm_tcpグループの作成 - サンプルコードの変更を取り消し

File: crane_plus_description/urdf/crane_plus.urdf.xacro (robot description, xacro)
@@ -66,5 +66,5 @@
     name_link_4="${NAME_LINK_4}"
     name_link_hand="${NAME_LINK_HAND}"
-    name_link_endtip="${NAME_LINK_ENDTIP}"
+    name_link_tcp="${NAME_LINK_TCP}"
     name_joint_base="${NAME_JOINT_BASE}"
     name_joint_1="${NAME_JOINT_1}"

File: crane_plus_description/urdf/crane_plus.xacro (robot description, xacro)
@@ -48,5 +48,5 @@
               name_joint_4
               name_joint_hand
-              name_joint_endtip
+              name_joint_tcp
               joints_vlimit
               joint_1_lower_limit
@@ -271,11 +271,10 @@
     </link>
     <!-- Tool Center Point for MoveIt -->
-    <joint name="${name_joint_endtip}" type="fixed">
+    <joint name="${name_joint_tcp}" type="fixed">
       <origin xyz="0 0 0.090" rpy="0 ${-M_PI/2} 0"/>
       <parent link="${name_link_4}"/>
-      <child link="${name_link_endtip}"/>
-    </joint>
-    <link name="${name_link_endtip}">
-    </link>
+      <child link="${name_link_tcp}"/>
+    </joint>
+    <link name="${name_link_tcp}"/>
     <!-- camera -->
     <xacro:if value="$(arg use_camera)">

Commit message: tcpの位置と姿勢のオフセットをローンチファイルの中で変更できるようにした．

File: crane_plus_description/urdf/crane_plus.urdf.xacro (robot description, xacro)
@@ -22,4 +22,6 @@
   <xacro:arg name="gz_control_config_package" default="" />
   <xacro:arg name="gz_control_config_file_path" default="" />
+  <xacro:arg name="tcp_offset_xyz" default="0 0 0" />
+  <xacro:arg name="tcp_offset_rpy" default="0 0 0" />
   <!-- Link to provide the location reference for the arm -->
   <link name="base_link"/>
@@ -85,5 +87,7 @@
     joint_hand_lower_limit="${JOINT_HAND_LOWER_LIMIT}"
     joint_hand_upper_limit="${JOINT_HAND_UPPER_LIMIT}"
-    use_camera="$(arg use_camera)">
+    use_camera="$(arg use_camera)"
+    tcp_offset_xyz="$(arg tcp_offset_xyz)"
+    tcp_offset_rpy="$(arg tcp_offset_rpy)">
     <origin xyz="0 0 0"/>
   </xacro:crane_plus>

File: crane_plus_description/urdf/crane_plus.xacro (robot description, xacro)
@@ -61,4 +61,6 @@
               joint_hand_upper_limit
               use_camera
+              tcp_offset_xyz
+              tcp_offset_rpy
               *origin">
     <joint name="${name_joint_base}" type="fixed">
@@ -272,5 +274,5 @@
     <!-- Tool Center Point for MoveIt -->
     <joint name="${name_joint_tcp}" type="fixed">
-      <origin xyz="0 0 0.090" rpy="0 ${-M_PI/2} 0"/>
+      <origin xyz="${tcp_offset_xyz}" rpy="${tcp_offset_rpy}"/>
       <parent link="${name_link_4}"/>
       <child link="${name_link_tcp}"/>

Commit message: base_linkとworldのジョイントをS17に合わせる

File: crane_plus_description/urdf/crane_plus.urdf.xacro (robot description, xacro)
@@ -17,12 +17,4 @@
   <xacro:arg name="gz_control_config_package" default="" />
   <xacro:arg name="gz_control_config_file_path" default="" />
-  <!-- Link to provide the location reference for the arm -->
-  <link name="base_link"/>
-  <!-- Used for fixing robot to Gazebo 'base_link' -->
-  <link name="world"/>
-  <joint name="base_link_to_world_joint" type="fixed">
-    <parent link="world"/>
-    <child link="base_link"/>
-  </joint>
   <xacro:property name="NAME_LINK_BASE" value="crane_plus_base"/>
   <xacro:property name="NAME_LINK_1" value="crane_plus_link1"/>
@@ -51,4 +43,11 @@
   <xacro:property name="JOINT_HAND_LOWER_LIMIT" value="${109.38 * TO_RADIAN - SERVO_HOME}"/>
   <xacro:property name="JOINT_HAND_UPPER_LIMIT" value="${188.27 * TO_RADIAN - SERVO_HOME}"/>
+  <!-- Used for fixing robot 'base_link' to Gazebo 'world' -->
+  <link name="world"/>
+  <link name="base_link"/>
+  <joint name="base_link_to_world_joint" type="fixed">
+    <parent link="world"/>
+    <child link="base_link"/>
+  </joint>
   <xacro:crane_plus
     parent="base_link"
