Commit message: 度数法から弧度法への変換にradians()を使用、effortの制限を変数に置き換える

File: crane_plus_description/urdf/crane_plus.urdf.xacro (robot description, xacro)
@@ -30,17 +30,17 @@
   <xacro:property name="NAME_JOINT_HAND" value="crane_plus_joint_hand"/>
   <xacro:property name="M_PI" value="3.14159"/>
-  <xacro:property name="TO_RADIAN" value="${M_PI / 180.0}"/>
-  <xacro:property name="SERVO_HOME" value="${TO_RADIAN * 150.0}"/>
+  <xacro:property name="SERVO_HOME" value="${radians(150.0)}"/>
+  <xacro:property name="JOINT_EFFORT_LIMIT" value="1.5"/>
   <xacro:property name="JOINT_VELOCITY_LIMIT" value="2.0"/>
-  <xacro:property name="JOINT_1_LOWER_LIMIT" value="${0.0 * TO_RADIAN - SERVO_HOME}"/>
-  <xacro:property name="JOINT_1_UPPER_LIMIT" value="${300.0 * TO_RADIAN - SERVO_HOME}"/>
-  <xacro:property name="JOINT_2_LOWER_LIMIT" value="${45.45 * TO_RADIAN - SERVO_HOME}"/>
-  <xacro:property name="JOINT_2_UPPER_LIMIT" value="${252.20 * TO_RADIAN - SERVO_HOME}"/>
-  <xacro:property name="JOINT_3_LOWER_LIMIT" value="${3.52 * TO_RADIAN - SERVO_HOME}"/>
-  <xacro:property name="JOINT_3_UPPER_LIMIT" value="${290.62 * TO_RADIAN - SERVO_HOME}"/>
-  <xacro:property name="JOINT_4_LOWER_LIMIT" value="${44.57 * TO_RADIAN - SERVO_HOME}"/>
-  <xacro:property name="JOINT_4_UPPER_LIMIT" value="${251.32 * TO_RADIAN - SERVO_HOME}"/>
-  <xacro:property name="JOINT_HAND_LOWER_LIMIT" value="${109.38 * TO_RADIAN - SERVO_HOME}"/>
-  <xacro:property name="JOINT_HAND_UPPER_LIMIT" value="${188.27 * TO_RADIAN - SERVO_HOME}"/>
+  <xacro:property name="JOINT_1_LOWER_LIMIT" value="${radians(0) - SERVO_HOME}"/>
+  <xacro:property name="JOINT_1_UPPER_LIMIT" value="${radians(300) - SERVO_HOME}"/>
+  <xacro:property name="JOINT_2_LOWER_LIMIT" value="${radians(46) - SERVO_HOME}"/>
+  <xacro:property name="JOINT_2_UPPER_LIMIT" value="${radians(252) - SERVO_HOME}"/>
+  <xacro:property name="JOINT_3_LOWER_LIMIT" value="${radians(4) - SERVO_HOME}"/>
+  <xacro:property name="JOINT_3_UPPER_LIMIT" value="${radians(290) - SERVO_HOME}"/>
+  <xacro:property name="JOINT_4_LOWER_LIMIT" value="${radians(45) - SERVO_HOME}"/>
+  <xacro:property name="JOINT_4_UPPER_LIMIT" value="${radians(251) - SERVO_HOME}"/>
+  <xacro:property name="JOINT_HAND_LOWER_LIMIT" value="${radians(110) - SERVO_HOME}"/>
+  <xacro:property name="JOINT_HAND_UPPER_LIMIT" value="${radians(188) - SERVO_HOME}"/>
   <!-- Used for fixing robot 'base_link' to Gazebo 'world' -->
   <link name="world"/>
@@ -64,4 +64,5 @@
     name_joint_4="${NAME_JOINT_4}"
     name_joint_hand="${NAME_JOINT_HAND}"
+    joints_elimit="${JOINT_EFFORT_LIMIT}"
     joints_vlimit="${JOINT_VELOCITY_LIMIT}"
     joint_1_lower_limit="${JOINT_1_LOWER_LIMIT}"

File: crane_plus_description/urdf/crane_plus.xacro (robot description, xacro)
@@ -21,4 +21,5 @@
               name_joint_4
               name_joint_hand
+              joints_elimit
               joints_vlimit
               joint_1_lower_limit
@@ -64,5 +65,5 @@
       <axis xyz="0 0 1"/>
       <limit
-        effort="1.5"
+        effort="${joints_elimit}"
         velocity="${joints_vlimit}"
         lower="${joint_1_lower_limit}"
@@ -98,5 +99,5 @@
       <axis xyz="0 1 0"/>
       <limit
-        effort="1.5"
+        effort="${joints_elimit}"
         velocity="${joints_vlimit}"
         lower="${joint_2_lower_limit}"
@@ -132,5 +133,5 @@
       <axis xyz="0 -1 0"/>
       <limit
-        effort="1.5"
+        effort="${joints_elimit}"
         velocity="${joints_vlimit}"
         lower="${joint_3_lower_limit}"
@@ -166,5 +167,5 @@
       <axis xyz="0 -1 0"/>
       <limit
-        effort="1.5"
+        effort="${joints_elimit}"
         velocity="${joints_vlimit}"
         lower="${joint_4_lower_limit}"
@@ -200,5 +201,5 @@
       <axis xyz="-1 0 0"/>
       <limit
-        effort="1.5"
+        effort="${joints_elimit}"
         velocity="${joints_vlimit}"
         lower="${joint_hand_lower_limit}"

Commit message: crane_plusマクロのパラメータを削除

File: crane_plus_description/urdf/crane_plus.urdf.xacro (robot description, xacro)
@@ -50,32 +50,6 @@
     <child link="base_link"/>
   </joint>
-  <xacro:crane_plus
-    parent="base_link"
-    name_link_base="${NAME_LINK_BASE}"
-    name_link_1="${NAME_LINK_1}"
-    name_link_2="${NAME_LINK_2}"
-    name_link_3="${NAME_LINK_3}"
-    name_link_4="${NAME_LINK_4}"
-    name_link_hand="${NAME_LINK_HAND}"
-    name_joint_base="${NAME_JOINT_BASE}"
-    name_joint_1="${NAME_JOINT_1}"
-    name_joint_2="${NAME_JOINT_2}"
-    name_joint_3="${NAME_JOINT_3}"
-    name_joint_4="${NAME_JOINT_4}"
-    name_joint_hand="${NAME_JOINT_HAND}"
-    joints_elimit="${JOINT_EFFORT_LIMIT}"
-    joints_vlimit="${JOINT_VELOCITY_LIMIT}"
-    joint_1_lower_limit="${JOINT_1_LOWER_LIMIT}"
-    joint_1_upper_limit="${JOINT_1_UPPER_LIMIT}"
-    joint_2_lower_limit="${JOINT_2_LOWER_LIMIT}"
-    joint_2_upper_limit="${JOINT_2_UPPER_LIMIT}"
-    joint_3_lower_limit="${JOINT_3_LOWER_LIMIT}"
-    joint_3_upper_limit="${JOINT_3_UPPER_LIMIT}"
-    joint_4_lower_limit="${JOINT_4_LOWER_LIMIT}"
-    joint_4_upper_limit="${JOINT_4_UPPER_LIMIT}"
-    joint_hand_lower_limit="${JOINT_HAND_LOWER_LIMIT}"
-    joint_hand_upper_limit="${JOINT_HAND_UPPER_LIMIT}"
-    use_camera="$(arg use_camera)">
-    <origin xyz="0 0 0"/>
+  <xacro:crane_plus parent="base_link">
+    <origin xyz="0 0 0" rpy="0 0 0"/>
   </xacro:crane_plus>
   <xacro:unless value="$(arg use_gazebo)">

File: crane_plus_description/urdf/crane_plus.xacro (robot description, xacro)
@@ -7,38 +7,11 @@
     <color rgba="0.95 0.95 0.95 1.0"/>
   </material>
-  <xacro:macro name="crane_plus"
-      params="parent
-              name_link_base
-              name_link_1
-              name_link_2
-              name_link_3
-              name_link_4
-              name_link_hand
-              name_joint_base
-              name_joint_1
-              name_joint_2
-              name_joint_3
-              name_joint_4
-              name_joint_hand
-              joints_elimit
-              joints_vlimit
-              joint_1_lower_limit
-              joint_1_upper_limit
-              joint_2_lower_limit
-              joint_2_upper_limit
-              joint_3_lower_limit
-              joint_3_upper_limit
-              joint_4_lower_limit
-              joint_4_upper_limit
-              joint_hand_lower_limit
-              joint_hand_upper_limit
-              use_camera
-              *origin">
-    <joint name="${name_joint_base}" type="fixed">
+  <xacro:macro name="crane_plus" params="parent *origin">
+    <joint name="${NAME_JOINT_BASE}" type="fixed">
       <xacro:insert_block name="origin"/>
       <parent link="${parent}"/>
-      <child link="${name_link_base}"/>
-    </joint>
-    <link name="${name_link_base}">
+      <child link="${NAME_LINK_BASE}"/>
+    </joint>
+    <link name="${NAME_LINK_BASE}">
       <visual>
         <origin xyz="0 0 0" rpy="0 0 0"/>
@@ -61,18 +34,18 @@
       </inertial>
     </link>
-    <joint name="${name_joint_1}" type="revolute">
+    <joint name="${NAME_JOINT_1}" type="revolute">
       <origin xyz="0 0 0.0454" rpy="0 0 0"/>
       <axis xyz="0 0 1"/>
       <limit
-        effort="${joints_elimit}"
-        velocity="${joints_vlimit}"
-        lower="${joint_1_lower_limit}"
-        upper="${joint_1_upper_limit}"
-        />
-      <parent link="${name_link_base}"/>
-      <child link="${name_link_1}"/>
-      <dynamics damping="1.0e-6" friction="2.0e-1"/>
-    </joint>
-    <link name="${name_link_1}">
+        effort="${JOINT_EFFORT_LIMIT}"
+        velocity="${JOINT_VELOCITY_LIMIT}"
+        lower="${JOINT_1_LOWER_LIMIT}"
+        upper="${JOINT_1_UPPER_LIMIT}"
+        />
+      <parent link="${NAME_LINK_BASE}"/>
+      <child link="${NAME_LINK_1}"/>
+      <dynamics damping="1.0e-6" friction="2.0e-1"/>
+    </joint>
+    <link name="${NAME_LINK_1}">
       <visual>
         <origin xyz="0 0 0" rpy="0 0 ${M_PI}"/>
@@ -95,18 +68,18 @@
       </inertial>
     </link>
-    <joint name="${name_joint_2}" type="revolute">
+    <joint name="${NAME_JOINT_2}" type="revolute">
       <origin xyz="0 0 0.026" rpy="0 0 0"/>
       <axis xyz="0 1 0"/>
       <limit
-        effort="${joints_elimit}"
-        velocity="${joints_vlimit}"
-        lower="${joint_2_lower_limit}"
-        upper="${joint_2_upper_limit}"
-        />
-      <parent link="${name_link_1}"/>
-      <child link="${name_link_2}"/>
-      <dynamics damping="1.0e-6" friction="2.0e-1"/>
-    </joint>
-    <link name="${name_link_2}">
+        effort="${JOINT_EFFORT_LIMIT}"
+        velocity="${JOINT_VELOCITY_LIMIT}"
+        lower="${JOINT_2_LOWER_LIMIT}"
+        upper="${JOINT_2_UPPER_LIMIT}"
+        />
+      <parent link="${NAME_LINK_1}"/>
+      <child link="${NAME_LINK_2}"/>
+      <dynamics damping="1.0e-6" friction="2.0e-1"/>
+    </joint>
+    <link name="${NAME_LINK_2}">
       <visual>
         <origin xyz="0 0 0" rpy="${M_PI/2} 0 0"/>
@@ -129,18 +102,18 @@
       </inertial>
     </link>
-    <joint name="${name_joint_3}" type="revolute">
+    <joint name="${NAME_JOINT_3}" type="revolute">
       <origin xyz="0 0 0.083" rpy="0 0 0"/>
       <axis xyz="0 -1 0"/>
       <limit
-        effort="${joints_elimit}"
-        velocity="${joints_vlimit}"
-        lower="${joint_3_lower_limit}"
-        upper="${joint_3_upper_limit}"
-        />
-      <parent link="${name_link_2}"/>
-      <child link="${name_link_3}"/>
-      <dynamics damping="1.0e-6" friction="2.0e-1"/>
-    </joint>
-    <link name="${name_link_3}">
+        effort="${JOINT_EFFORT_LIMIT}"
+        velocity="${JOINT_VELOCITY_LIMIT}"
+        lower="${JOINT_3_LOWER_LIMIT}"
+        upper="${JOINT_3_UPPER_LIMIT}"
+        />
+      <parent link="${NAME_LINK_2}"/>
+      <child link="${NAME_LINK_3}"/>
+      <dynamics damping="1.0e-6" friction="2.0e-1"/>
+    </joint>
+    <link name="${NAME_LINK_3}">
       <visual>
         <origin xyz="0 0 0" rpy="${M_PI/2} 0 0"/>
@@ -163,18 +136,18 @@
       </inertial>
     </link>
-    <joint name="${name_joint_4}" type="revolute">
+    <joint name="${NAME_JOINT_4}" type="revolute">
       <origin xyz="0 0 0.0935" rpy="0 0 0"/>
       <axis xyz="0 -1 0"/>
       <limit
-        effort="${joints_elimit}"
-        velocity="${joints_vlimit}"
-        lower="${joint_4_lower_limit}"
-        upper="${joint_4_upper_limit}"
-        />
-      <parent link="${name_link_3}"/>
-      <child link="${name_link_4}"/>
-      <dynamics damping="1.0e-6" friction="2.0e-1"/>
-    </joint>
-    <link name="${name_link_4}">
+        effort="${JOINT_EFFORT_LIMIT}"
+        velocity="${JOINT_VELOCITY_LIMIT}"
+        lower="${JOINT_4_LOWER_LIMIT}"
+        upper="${JOINT_4_UPPER_LIMIT}"
+        />
+      <parent link="${NAME_LINK_3}"/>
+      <child link="${NAME_LINK_4}"/>
+      <dynamics damping="1.0e-6" friction="2.0e-1"/>
+    </joint>
+    <link name="${NAME_LINK_4}">
       <visual>
         <origin xyz="0 0 0" rpy="${M_PI/2} 0 0"/>
@@ -197,18 +170,18 @@
       </inertial>
     </link>
-    <joint name="${name_joint_hand}" type="revolute">
+    <joint name="${NAME_JOINT_HAND}" type="revolute">
       <origin xyz="0 -0.0145 0.045" rpy="0 0 0"/>
       <axis xyz="-1 0 0"/>
       <limit
-        effort="${joints_elimit}"
-        velocity="${joints_vlimit}"
-        lower="${joint_hand_lower_limit}"
-        upper="${joint_hand_upper_limit}"
-        />
-      <parent link="${name_link_4}"/>
-      <child link="${name_link_hand}"/>
-      <dynamics damping="1.0e-6" friction="2.0e-1"/>
-    </joint>
-    <link name="${name_link_hand}">
+        effort="${JOINT_EFFORT_LIMIT}"
+        velocity="${JOINT_VELOCITY_LIMIT}"
+        lower="${JOINT_HAND_LOWER_LIMIT}"
+        upper="${JOINT_HAND_UPPER_LIMIT}"
+        />
+      <parent link="${NAME_LINK_4}"/>
+      <child link="${NAME_LINK_HAND}"/>
+      <dynamics damping="1.0e-6" friction="2.0e-1"/>
+    </joint>
+    <link name="${NAME_LINK_HAND}">
       <visual>
         <origin xyz="0 0 0" rpy="0 -${M_PI/2} 0"/>

Commit message: 実機の動作に合わせて関節角度の制限を広げる

File: crane_plus_description/urdf/crane_plus.urdf.xacro (robot description, xacro)
@@ -55,12 +55,12 @@
   <xacro:property name="JOINT_1_LOWER_LIMIT" value="${radians(0) - SERVO_HOME}"/>
   <xacro:property name="JOINT_1_UPPER_LIMIT" value="${radians(300) - SERVO_HOME}"/>
-  <xacro:property name="JOINT_2_LOWER_LIMIT" value="${radians(46) - SERVO_HOME}"/>
-  <xacro:property name="JOINT_2_UPPER_LIMIT" value="${radians(252) - SERVO_HOME}"/>
-  <xacro:property name="JOINT_3_LOWER_LIMIT" value="${radians(4) - SERVO_HOME}"/>
-  <xacro:property name="JOINT_3_UPPER_LIMIT" value="${radians(290) - SERVO_HOME}"/>
-  <xacro:property name="JOINT_4_LOWER_LIMIT" value="${radians(45) - SERVO_HOME}"/>
-  <xacro:property name="JOINT_4_UPPER_LIMIT" value="${radians(251) - SERVO_HOME}"/>
-  <xacro:property name="JOINT_HAND_LOWER_LIMIT" value="${radians(110) - SERVO_HOME}"/>
-  <xacro:property name="JOINT_HAND_UPPER_LIMIT" value="${radians(188) - SERVO_HOME}"/>
+  <xacro:property name="JOINT_2_LOWER_LIMIT" value="${radians(45) - SERVO_HOME}"/>
+  <xacro:property name="JOINT_2_UPPER_LIMIT" value="${radians(253) - SERVO_HOME}"/>
+  <xacro:property name="JOINT_3_LOWER_LIMIT" value="${radians(3) - SERVO_HOME}"/>
+  <xacro:property name="JOINT_3_UPPER_LIMIT" value="${radians(291) - SERVO_HOME}"/>
+  <xacro:property name="JOINT_4_LOWER_LIMIT" value="${radians(44) - SERVO_HOME}"/>
+  <xacro:property name="JOINT_4_UPPER_LIMIT" value="${radians(252) - SERVO_HOME}"/>
+  <xacro:property name="JOINT_HAND_LOWER_LIMIT" value="${radians(109) - SERVO_HOME}"/>
+  <xacro:property name="JOINT_HAND_UPPER_LIMIT" value="${radians(189) - SERVO_HOME}"/>
   <!-- Used for fixing robot 'base_link' to Gazebo 'world' -->
   <link name="world"/>

Commit message: 円周率の変数M_PIを削除してradians()を使用

File: crane_plus_description/urdf/crane_plus.urdf.xacro (robot description, xacro)
@@ -49,5 +49,4 @@
   <xacro:property name="NAME_JOINT_4" value="crane_plus_joint4"/>
   <xacro:property name="NAME_JOINT_HAND" value="crane_plus_joint_hand"/>
-  <xacro:property name="M_PI" value="3.14159"/>
   <xacro:property name="SERVO_HOME" value="${radians(150.0)}"/>
   <xacro:property name="JOINT_EFFORT_LIMIT" value="1.5"/>

File: crane_plus_description/urdf/crane_plus.xacro (robot description, xacro)
@@ -43,5 +43,5 @@
     <link name="${NAME_LINK_1}">
       <visual>
-        <origin xyz="0 0 0" rpy="0 0 ${M_PI}"/>
+        <origin xyz="0 0 0" rpy="0 0 0"/>
         <geometry>
           <mesh filename="package://crane_plus_description/meshes/visual/Link1_20201013.stl" scale="1 1 1"/>
@@ -50,5 +50,5 @@
       </visual>
       <collision>
-        <origin xyz="0 0 0" rpy="0 0 ${M_PI}"/>
+        <origin xyz="0 0 0" rpy="0 0 0"/>
         <geometry>
           <mesh filename="package://crane_plus_description/meshes/collision/Link1_collision_20201013.stl" scale="1 1 1"/>
@@ -77,5 +77,5 @@
     <link name="${NAME_LINK_2}">
       <visual>
-        <origin xyz="0 0 0" rpy="${M_PI/2} 0 0"/>
+        <origin xyz="0 0 0" rpy="${radians(90)} 0 0"/>
         <geometry>
           <mesh filename="package://crane_plus_description/meshes/visual/Link2_20201013.stl" scale="1 1 1"/>
@@ -84,5 +84,5 @@
       </visual>
       <collision>
-        <origin xyz="0 0 0" rpy="${M_PI/2} 0 0"/>
+        <origin xyz="0 0 0" rpy="${radians(90)} 0 0"/>
         <geometry>
           <mesh filename="package://crane_plus_description/meshes/collision/Link2_collision_20201013.stl" scale="1 1 1"/>
@@ -92,5 +92,5 @@
       <inertial>
         <mass value="1.17E-01"/>
-        <origin xyz="7.99E-04 1.00E-06 4.15E-02" rpy="${M_PI/2} 0 0"/>
+        <origin xyz="7.99E-04 1.00E-06 4.15E-02" rpy="${radians(90)} 0 0"/>
         <inertia ixx="1.25E-04" ixy="6.83E-08" ixz="9.50E-11" iyy="1.92E-05" iyz="0.0" izz="1.19E-04"/>
       </inertial>
@@ -111,5 +111,5 @@
     <link name="${NAME_LINK_3}">
       <visual>
-        <origin xyz="0 0 0" rpy="${M_PI/2} 0 0"/>
+        <origin xyz="0 0 0" rpy="${radians(90)} 0 0"/>
         <geometry>
           <mesh filename="package://crane_plus_description/meshes/visual/Link3_20201013.stl" scale="1 1 1"/>
@@ -118,5 +118,5 @@
       </visual>
       <collision>
-        <origin xyz="0 0 0" rpy="${M_PI/2} 0 0"/>
+        <origin xyz="0 0 0" rpy="${radians(90)} 0 0"/>
         <geometry>
           <mesh filename="package://crane_plus_description/meshes/collision/Link3_collision_20201013.stl" scale="1 1 1"/>
@@ -126,5 +126,5 @@
       <inertial>
         <mass value="7.23E-02"/>
-        <origin xyz="6.45E-04 -1.38E-04 7.01E-02" rpy="${M_PI/2} 0 0"/>
+        <origin xyz="6.45E-04 -1.38E-04 7.01E-02" rpy="${radians(90)} 0 0"/>
         <inertia ixx="5.41E-05" ixy="-2.28E-07" ixz="-2.67E-09" iyy="1.60E-05" iyz="-5.35E-07" izz="4.69E-05"/>
       </inertial>
@@ -145,5 +145,5 @@
     <link name="${NAME_LINK_4}">
       <visual>
-        <origin xyz="0 0 0" rpy="${M_PI/2} 0 0"/>
+        <origin xyz="0 0 0" rpy="${radians(90)} 0 0"/>
         <geometry>
           <mesh filename="package://crane_plus_description/meshes/visual/Link4_20201013.stl" scale="1 1 1"/>
@@ -152,5 +152,5 @@
       </visual>
       <collision>
-        <origin xyz="0 0 0" rpy="${M_PI/2} 0 0"/>
+        <origin xyz="0 0 0" rpy="${radians(90)} 0 0"/>
         <geometry>
           <mesh filename="package://crane_plus_description/meshes/collision/Link4_collision_20201013.stl" scale="1 1 1"/>
@@ -160,5 +160,5 @@
       <inertial>
         <mass value="8.19E-02"/>
-        <origin xyz="6.45E-04 -5.70E-04 4.62E-02" rpy="${M_PI/2} 0 0"/>
+        <origin xyz="6.45E-04 -5.70E-04 4.62E-02" rpy="${radians(90)} 0 0"/>
         <inertia ixx="5.91E-05" ixy="-5.11E-08" ixz="3.49E-07" iyy="3.62E-05" iyz="1.37E-05" izz="3.98E-05"/>
       </inertial>
@@ -179,5 +179,5 @@
     <link name="${NAME_LINK_HAND}">
       <visual>
-        <origin xyz="0 0 0" rpy="0 -${M_PI/2} 0"/>
+        <origin xyz="0 0 0" rpy="0 ${radians(-90)} 0"/>
         <geometry>
           <mesh filename="package://crane_plus_description/meshes/visual/Hand_20201013.stl" scale="1 1 1"/>
@@ -186,5 +186,5 @@
       </visual>
       <collision>
-        <origin xyz="0 0 0" rpy="0 -${M_PI/2} 0"/>
+        <origin xyz="0 0 0" rpy="0 ${radians(-90)} 0"/>
         <geometry>
           <mesh filename="package://crane_plus_description/meshes/collision/Hand_collision_20201013.stl" scale="1 1 1"/>
@@ -194,5 +194,5 @@
       <inertial>
         <mass value="2.29E-02"/>
-        <origin xyz="0.0 -2.04E-02 2.77E-02" rpy="0 -${M_PI/2} 0"/>
+        <origin xyz="0.0 -2.04E-02 2.77E-02" rpy="0 ${radians(-90)} 0"/>
         <inertia ixx="5.76E-06" ixy="-4.66E-07" ixz="0.0" iyy="2.76E-05" iyz="0.0" izz="2.52E-05"/>
       </inertial>

Commit message: TCPリンクを追加

File: crane_plus_description/urdf/crane_plus.urdf.xacro (robot description, xacro)
@@ -43,4 +43,5 @@
   <xacro:property name="NAME_LINK_4" value="crane_plus_link4"/>
   <xacro:property name="NAME_LINK_HAND" value="crane_plus_link_hand"/>
+  <xacro:property name="NAME_LINK_TCP" value="crane_plus_link_TCP"/>
   <xacro:property name="NAME_JOINT_BASE" value="crane_plus_joint_base"/>
   <xacro:property name="NAME_JOINT_1" value="crane_plus_joint1"/>
@@ -49,4 +50,5 @@
   <xacro:property name="NAME_JOINT_4" value="crane_plus_joint4"/>
   <xacro:property name="NAME_JOINT_HAND" value="crane_plus_joint_hand"/>
+  <xacro:property name="NAME_JOINT_TCP" value="crane_plus_joint_tcp"/>
   <xacro:property name="SERVO_HOME" value="${radians(150.0)}"/>
   <xacro:property name="JOINT_EFFORT_LIMIT" value="1.5"/>

File: crane_plus_description/urdf/crane_plus.xacro (robot description, xacro)
@@ -198,4 +198,10 @@
       </inertial>
     </link>
+    <joint name="${NAME_JOINT_TCP}" type="fixed">
+      <origin xyz="0 0 0.09" rpy="0 0 0"/>
+      <parent link="${NAME_LINK_4}"/>
+      <child link="${NAME_LINK_TCP}"/>
+    </joint>
+    <link name="${NAME_LINK_TCP}"/>
   </xacro:macro>
 </robot>

Commit message: リンク名を小文字に統一

File: crane_plus_description/urdf/crane_plus.urdf.xacro (robot description, xacro)
@@ -43,5 +43,5 @@
   <xacro:property name="NAME_LINK_4" value="crane_plus_link4"/>
   <xacro:property name="NAME_LINK_HAND" value="crane_plus_link_hand"/>
-  <xacro:property name="NAME_LINK_TCP" value="crane_plus_link_TCP"/>
+  <xacro:property name="NAME_LINK_TCP" value="crane_plus_link_tcp"/>
   <xacro:property name="NAME_JOINT_BASE" value="crane_plus_joint_base"/>
   <xacro:property name="NAME_JOINT_1" value="crane_plus_joint1"/>
