Commit message: fix joint origin

File: crane_plus_description/urdf/crane_plus.xacro (robot description, xacro)
@@ -100,5 +100,5 @@
     <joint name="${NAME_JOINT_2}" type="revolute">
       <origin xyz="0 0 0.026" rpy="0 0 0"/>
-      <axis xyz="0 -1 0"/>
+      <axis xyz="0 1 0"/>
       <limit
         effort="10.0"
@@ -129,5 +129,5 @@
     <joint name="${NAME_JOINT_3}" type="revolute">
       <origin xyz="0 0 0.083" rpy="0 0 0"/>
-      <axis xyz="0 1 0"/>
+      <axis xyz="0 -1 0"/>
       <limit
         effort="10.0"
@@ -186,6 +186,6 @@
     </link>
     <joint name="${NAME_JOINT_HAND}" type="revolute">
-      <origin xyz="0 0 0.045" rpy="0 0 0"/>
-      <axis xyz="1 0 0"/>
+      <origin xyz="0 -0.0145 0.045" rpy="0 0 0"/>
+      <axis xyz="-1 0 0"/>
       <limit
         effort="10.0"
@@ -200,5 +200,5 @@
     <link name="${NAME_LINK_HAND}">
       <visual>
-        <origin xyz="0 -0.0145 0" rpy="0 -${M_PI/2} 0"/>
+        <origin xyz="0 0 0" rpy="0 -${M_PI/2} 0"/>
         <geometry>
           <mesh filename="package://crane_plus_description/meshes/visual/RT-CRANE+_Hand.stl"

Commit message: Fix collision model

File: crane_plus_description/urdf/crane_plus.xacro (robot description, xacro)
@@ -62,7 +62,7 @@
       </visual>
       <collision>
-        <origin xyz="0 0 0" rpy="0 0 0"/>
-        <geometry>
-          <box size="0.01 0.02 0.04"/>
+        <origin xyz="-0.0145 0 0.02" rpy="0 0 0"/>
+        <geometry>
+          <box size="0.0485 0.0255 0.032"/>
         </geometry>
       </collision>
@@ -91,7 +91,7 @@
       </visual>
       <collision>
-        <origin xyz="0 0 0" rpy="0 0 0"/>
-        <geometry>
-          <box size="0.01 0.02 0.04"/>
+        <origin xyz="0 0 0.0035" rpy="0 0 0"/>
+        <geometry>
+          <box size="0.0245 0.048 0.003"/>
         </geometry>
       </collision>
@@ -120,7 +120,7 @@
       </visual>
       <collision>
-        <origin xyz="0 0 0" rpy="0 0 0"/>
-        <geometry>
-          <box size="0.01 0.02 0.04"/>
+        <origin xyz="0 0 0.040" rpy="0 0 0"/>
+        <geometry>
+          <box size="0.0315 0.038 0.105"/>
         </geometry>
       </collision>
@@ -149,7 +149,7 @@
       </visual>
       <collision>
-        <origin xyz="0 0 0" rpy="0 0 0"/>
-        <geometry>
-          <box size="0.01 0.02 0.04"/>
+        <origin xyz="0 0 0.08" rpy="0 0 0"/>
+        <geometry>
+          <box size="0.032 0.035 0.050"/>
         </geometry>
       </collision>
@@ -178,7 +178,7 @@
       </visual>
       <collision>
-        <origin xyz="0 0 0" rpy="${M_PI/2} 0 0"/>
-        <geometry>
-          <box size="0.01 0.02 0.04"/>
+        <origin xyz="0 0.037 0.097" rpy="${M_PI/2} 0 0"/>
+        <geometry>
+          <box size="0.034 0.045 0.002"/>
         </geometry>
       </collision>
@@ -207,7 +207,7 @@
       </visual>
       <collision>
-        <origin xyz="0 0 0" rpy="0 0 0"/>
-        <geometry>
-          <box size="0.01 0.02 0.04"/>
+        <origin xyz="0 -0.018 0.075" rpy="${M_PI/3} 0 0"/>
+        <geometry>
+          <box size="0.034 0.045 0.002"/>
         </geometry>
       </collision>

Commit message: Update xacro (#1)
* fix joint origin

* Fix joint limits

* Fix collision model

File: crane_plus_description/urdf/crane_plus.xacro (robot description, xacro)
@@ -19,5 +19,4 @@
     <color rgba="0.3 0.3 1.0 1.0"/>
   </material>
-  <xacro:property name="M_PI" value="3.14159"/>
   <xacro:property name="SCALE_MM" value="0.001"/>
   <xacro:property name="SCALE_CM" value="0.01"/>
@@ -63,7 +62,7 @@
       </visual>
       <collision>
-        <origin xyz="0 0 0" rpy="0 0 0"/>
-        <geometry>
-          <box size="0.01 0.02 0.04"/>
+        <origin xyz="-0.0145 0 0.02" rpy="0 0 0"/>
+        <geometry>
+          <box size="0.0485 0.0255 0.032"/>
         </geometry>
       </collision>
@@ -92,7 +91,7 @@
       </visual>
       <collision>
-        <origin xyz="0 0 0" rpy="0 0 0"/>
-        <geometry>
-          <box size="0.01 0.02 0.04"/>
+        <origin xyz="0 0 0.0035" rpy="0 0 0"/>
+        <geometry>
+          <box size="0.0245 0.048 0.003"/>
         </geometry>
       </collision>
@@ -100,5 +99,5 @@
     <joint name="${NAME_JOINT_2}" type="revolute">
       <origin xyz="0 0 0.026" rpy="0 0 0"/>
-      <axis xyz="0 -1 0"/>
+      <axis xyz="0 1 0"/>
       <limit
         effort="10.0"
@@ -121,7 +120,7 @@
       </visual>
       <collision>
-        <origin xyz="0 0 0" rpy="0 0 0"/>
-        <geometry>
-          <box size="0.01 0.02 0.04"/>
+        <origin xyz="0 0 0.040" rpy="0 0 0"/>
+        <geometry>
+          <box size="0.0315 0.038 0.105"/>
         </geometry>
       </collision>
@@ -129,5 +128,5 @@
     <joint name="${NAME_JOINT_3}" type="revolute">
       <origin xyz="0 0 0.083" rpy="0 0 0"/>
-      <axis xyz="0 1 0"/>
+      <axis xyz="0 -1 0"/>
       <limit
         effort="10.0"
@@ -150,7 +149,7 @@
       </visual>
       <collision>
-        <origin xyz="0 0 0" rpy="0 0 0"/>
-        <geometry>
-          <box size="0.01 0.02 0.04"/>
+        <origin xyz="0 0 0.08" rpy="0 0 0"/>
+        <geometry>
+          <box size="0.032 0.035 0.050"/>
         </geometry>
       </collision>
@@ -179,13 +178,13 @@
       </visual>
       <collision>
-        <origin xyz="0 0 0" rpy="${M_PI/2} 0 0"/>
-        <geometry>
-          <box size="0.01 0.02 0.04"/>
+        <origin xyz="0 0.037 0.097" rpy="${M_PI/2} 0 0"/>
+        <geometry>
+          <box size="0.034 0.045 0.002"/>
         </geometry>
       </collision>
     </link>
     <joint name="${NAME_JOINT_HAND}" type="revolute">
-      <origin xyz="0 0 0.045" rpy="0 0 0"/>
-      <axis xyz="1 0 0"/>
+      <origin xyz="0 -0.0145 0.045" rpy="0 0 0"/>
+      <axis xyz="-1 0 0"/>
       <limit
         effort="10.0"
@@ -200,5 +199,5 @@
     <link name="${NAME_LINK_HAND}">
       <visual>
-        <origin xyz="0 -0.0145 0" rpy="0 -${M_PI/2} 0"/>
+        <origin xyz="0 0 0" rpy="0 -${M_PI/2} 0"/>
         <geometry>
           <mesh filename="package://crane_plus_description/meshes/visual/RT-CRANE+_Hand.stl"
@@ -208,7 +207,7 @@
       </visual>
       <collision>
-        <origin xyz="0 0 0" rpy="0 0 0"/>
-        <geometry>
-          <box size="0.01 0.02 0.04"/>
+        <origin xyz="0 -0.018 0.075" rpy="${M_PI/3} 0 0"/>
+        <geometry>
+          <box size="0.034 0.045 0.002"/>
         </geometry>
       </collision>

Commit message: update inerital of URDF

File: crane_plus_description/urdf/crane_plus.xacro (robot description, xacro)
@@ -68,6 +68,7 @@
       </collision>
       <inertial>
-        <mass value="1"/>
-        <inertia ixx="1" ixy="0.0" ixz="0.0" iyy="1" iyz="0.0" izz="1"/>
+        <mass value="0.06645"/>
+        <origin xyz="-1.31E-02 7.00E-06 2.12E-02" rpy="0 ${M_PI/8} 0"/>
+        <inertia ixx="1.66E-05" ixy="1.80E-09" ixz="-5.75E-07" iyy="2.36E-05" iyz="-3.23E-08" izz="1.77E-05"/>
       </inertial>
     </link>
@@ -101,6 +102,7 @@
       </collision>
       <inertial>
-        <mass value="1"/>
-        <inertia ixx="1" ixy="0.0" ixz="0.0" iyy="1" iyz="0.0" izz="1"/>
+        <mass value="0.007729"/>
+        <origin xyz="2.00E-06 0.0 1.09E-02" rpy="0 0 0"/>
+        <inertia ixx="3.43E-06" ixy="0.0" ixz="1.66E-10" iyy="1.30E-06" iyz="0.0" izz="3.05E-06"/>
       </inertial>
     </link>
@@ -134,6 +136,7 @@
       </collision>
       <inertial>
-        <mass value="1"/>
-        <inertia ixx="1" ixy="0.0" ixz="0.0" iyy="1" iyz="0.0" izz="1"/>
+        <mass value="0.116745"/>
+        <origin xyz="7.99E-04 1.00E-06 4.15E-02" rpy="${M_PI/2} 0 0"/>
+        <inertia ixx="1.25E-04" ixy="6.83E-08" ixz="9.50E-11" iyy="1.92E-05" iyz="0.0" izz="1.19E-04"/>
       </inertial>
     </link>
@@ -167,6 +170,7 @@
       </collision>
       <inertial>
-        <mass value="1"/>
-        <inertia ixx="1" ixy="0.0" ixz="0.0" iyy="1" iyz="0.0" izz="1"/>
+        <mass value="0.072317"/>
+        <origin xyz="6.45E-04 -1.38E-04 7.01E-02" rpy="${M_PI/2} 0 0"/>
+        <inertia ixx="5.41E-05" ixy="-2.28E-07" ixz="-2.67E-09" iyy="1.60E-05" iyz="-5.35E-07" izz="4.69E-05"/>
       </inertial>
     </link>
@@ -200,6 +204,7 @@
       </collision>
       <inertial>
-        <mass value="1"/>
-        <inertia ixx="1" ixy="0.0" ixz="0.0" iyy="1" iyz="0.0" izz="1"/>
+        <mass value="0.08185"/>
+        <origin xyz="6.45E-04 -5.70E-04 4.62E-02" rpy="${M_PI/2} 0 0"/>
+        <inertia ixx="5.91E-05" ixy="-5.11E-08" ixz="3.49E-07" iyy="3.62E-05" iyz="1.37E-05" izz="3.98E-05"/>
       </inertial>
     </link>
@@ -233,6 +238,7 @@
       </collision>
       <inertial>
-        <mass value="1"/>
-        <inertia ixx="1" ixy="0.0" ixz="0.0" iyy="1" iyz="0.0" izz="1"/>
+        <mass value="0.022901"/>
+        <origin xyz="0.0 -2.04E-02 2.77E-02" rpy="0 ${M_PI/2} 0"/>
+        <inertia ixx="5.76E-06" ixy="-4.66E-07" ixz="0.0" iyy="2.76E-05" iyz="0.0" izz="2.52E-05"/>
       </inertial>
     </link>

Commit message: Add crane_plus_gazebo (#5)
* Add crane_plus_gazebo. Spawn CRANE+ and table and box

* update inerital of URDF

* Fix entity name

* Fix crane_plus.srdf

File: crane_plus_description/urdf/crane_plus.xacro (robot description, xacro)
@@ -27,5 +27,5 @@
   <xacro:property name="NAME_JOINT_4" value="crane_plus_joint4"/>
   <xacro:property name="NAME_JOINT_HAND" value="crane_plus_joint_hand"/>
-  <xacro:property name="NAME_LINK_BASE" value="base_link"/>
+  <xacro:property name="NAME_LINK_BASE" value="crane_plus_base"/>
   <xacro:property name="NAME_LINK_1" value="crane_plus_link1"/>
   <xacro:property name="NAME_LINK_2" value="crane_plus_link2"/>
@@ -47,9 +47,9 @@
               joint_hand_upper_limit
               *origin">
-    <!-- <joint name="${NAME_JOINT_BASE}" type="fixed"> -->
-    <!--   <xacro:insert_block name="origin"/>          -->
-    <!--   <parent link="${parent}"/>                   -->
-    <!--   <child link="${NAME_LINK_BASE}"/>            -->
-    <!-- </joint>                                       -->
+    <joint name="${NAME_JOINT_BASE}" type="fixed">
+      <xacro:insert_block name="origin"/>
+      <parent link="${parent}"/>
+      <child link="${NAME_LINK_BASE}"/>
+    </joint>
     <link name="${NAME_LINK_BASE}">
       <visual>
@@ -67,4 +67,9 @@
         </geometry>
       </collision>
+      <inertial>
+        <mass value="0.06645"/>
+        <origin xyz="-1.31E-02 7.00E-06 2.12E-02" rpy="0 ${M_PI/8} 0"/>
+        <inertia ixx="1.66E-05" ixy="1.80E-09" ixz="-5.75E-07" iyy="2.36E-05" iyz="-3.23E-08" izz="1.77E-05"/>
+      </inertial>
     </link>
     <joint name="${NAME_JOINT_1}" type="revolute">
@@ -96,4 +101,9 @@
         </geometry>
       </collision>
+      <inertial>
+        <mass value="0.007729"/>
+        <origin xyz="2.00E-06 0.0 1.09E-02" rpy="0 0 0"/>
+        <inertia ixx="3.43E-06" ixy="0.0" ixz="1.66E-10" iyy="1.30E-06" iyz="0.0" izz="3.05E-06"/>
+      </inertial>
     </link>
     <joint name="${NAME_JOINT_2}" type="revolute">
@@ -125,4 +135,9 @@
         </geometry>
       </collision>
+      <inertial>
+        <mass value="0.116745"/>
+        <origin xyz="7.99E-04 1.00E-06 4.15E-02" rpy="${M_PI/2} 0 0"/>
+        <inertia ixx="1.25E-04" ixy="6.83E-08" ixz="9.50E-11" iyy="1.92E-05" iyz="0.0" izz="1.19E-04"/>
+      </inertial>
     </link>
     <joint name="${NAME_JOINT_3}" type="revolute">
@@ -154,4 +169,9 @@
         </geometry>
       </collision>
+      <inertial>
+        <mass value="0.072317"/>
+        <origin xyz="6.45E-04 -1.38E-04 7.01E-02" rpy="${M_PI/2} 0 0"/>
+        <inertia ixx="5.41E-05" ixy="-2.28E-07" ixz="-2.67E-09" iyy="1.60E-05" iyz="-5.35E-07" izz="4.69E-05"/>
+      </inertial>
     </link>
     <joint name="${NAME_JOINT_4}" type="revolute">
@@ -183,4 +203,9 @@
         </geometry>
       </collision>
+      <inertial>
+        <mass value="0.08185"/>
+        <origin xyz="6.45E-04 -5.70E-04 4.62E-02" rpy="${M_PI/2} 0 0"/>
+        <inertia ixx="5.91E-05" ixy="-5.11E-08" ixz="3.49E-07" iyy="3.62E-05" iyz="1.37E-05" izz="3.98E-05"/>
+      </inertial>
     </link>
     <joint name="${NAME_JOINT_HAND}" type="revolute">
@@ -212,4 +237,9 @@
         </geometry>
       </collision>
+      <inertial>
+        <mass value="0.022901"/>
+        <origin xyz="0.0 -2.04E-02 2.77E-02" rpy="0 ${M_PI/2} 0"/>
+        <inertia ixx="5.76E-06" ixy="-4.66E-07" ixz="0.0" iyy="2.76E-05" iyz="0.0" izz="2.52E-05"/>
+      </inertial>
     </link>
   </xacro:macro>

Commit message: Update mesh data

File: crane_plus_description/urdf/crane_plus.xacro (robot description, xacro)
@@ -33,4 +33,16 @@
   <xacro:property name="NAME_LINK_4" value="crane_plus_link4"/>
   <xacro:property name="NAME_LINK_HAND" value="crane_plus_link_hand"/>
+  <xacro:property name="MESH_LINK_BASE" value="crane_plus_description/meshes/visual/body_20201013.stl"/>
+  <xacro:property name="MESH_LINK_1" value="crane_plus_description/meshes/visual/Link1_20201013.stl"/>
+  <xacro:property name="MESH_LINK_2" value="crane_plus_description/meshes/visual/Link2_20201013.stl"/>
+  <xacro:property name="MESH_LINK_3" value="crane_plus_description/meshes/visual/Link3_20201013.stl"/>
+  <xacro:property name="MESH_LINK_4" value="crane_plus_description/meshes/visual/Link4_20201013.stl"/>
+  <xacro:property name="MESH_LINK_HAND" value="crane_plus_description/meshes/visual/Hand_20201013.stl"/>
+  <xacro:property name="MESH_COLLISION_LINK_BASE" value="crane_plus_description/meshes/collision/body_collision_20201013.stl"/>
+  <xacro:property name="MESH_COLLISION_LINK_1" value="crane_plus_description/meshes/collision/Link1_collision_20201013.stl"/>
+  <xacro:property name="MESH_COLLISION_LINK_2" value="crane_plus_description/meshes/collision/Link2_collision_20201013.stl"/>
+  <xacro:property name="MESH_COLLISION_LINK_3" value="crane_plus_description/meshes/collision/Link3_collision_20201013.stl"/>
+  <xacro:property name="MESH_COLLISION_LINK_4" value="crane_plus_description/meshes/collision/Link4_collision_20201013.stl"/>
+  <xacro:property name="MESH_COLLISION_LINK_HAND" value="crane_plus_description/meshes/collision/Hand_collision_20201013.stl"/>
   <xacro:macro name="crane_plus"
       params="parent
@@ -56,14 +68,16 @@
         <origin xyz="0 0 0" rpy="0 0 0"/>
         <geometry>
-          <mesh filename="package://crane_plus_description/meshes/visual/RT-CRANE+_body.stl"
-              scale="1 1 1"/>
-        </geometry>
-        <material name="black"/>
-      </visual>
-      <collision>
-        <origin xyz="-0.0145 0 0.02" rpy="0 0 0"/>
-        <geometry>
-          <box size="0.0485 0.0255 0.032"/>
-        </geometry>
+          <mesh filename="package://${MESH_LINK_BASE}"
+              scale="1 1 1"/>
+        </geometry>
+        <material name="black"/>
+      </visual>
+      <collision>
+        <origin xyz="0 0 0" rpy="0 0 0"/>
+        <geometry>
+          <mesh filename="package://${MESH_COLLISION_LINK_BASE}"
+              scale="1 1 1"/>
+        </geometry>
+        <material name="black"/>
       </collision>
       <inertial>
@@ -90,14 +104,16 @@
         <origin xyz="0 0 0" rpy="0 0 ${M_PI}"/>
         <geometry>
-          <mesh filename="package://crane_plus_description/meshes/visual/RT-CRANE+_Link1.stl"
-              scale="1 1 1"/>
-        </geometry>
-        <material name="white"/>
-      </visual>
-      <collision>
-        <origin xyz="0 0 0.0035" rpy="0 0 0"/>
-        <geometry>
-          <box size="0.0245 0.048 0.003"/>
-        </geometry>
+          <mesh filename="package://${MESH_LINK_1}"
+              scale="1 1 1"/>
+        </geometry>
+        <material name="white"/>
+      </visual>
+      <collision>
+        <origin xyz="0 0 0" rpy="0 0 ${M_PI}"/>
+        <geometry>
+          <mesh filename="package://${MESH_COLLISION_LINK_1}"
+              scale="1 1 1"/>
+        </geometry>
+        <material name="white"/>
       </collision>
       <inertial>
@@ -124,14 +140,16 @@
         <origin xyz="0 0 0" rpy="${M_PI/2} 0 0"/>
         <geometry>
-          <mesh filename="package://crane_plus_description/meshes/visual/RT-CRANE+_Link2.stl"
-              scale="1 1 1"/>
-        </geometry>
-        <material name="black"/>
-      </visual>
-      <collision>
-        <origin xyz="0 0 0.040" rpy="0 0 0"/>
-        <geometry>
-          <box size="0.0315 0.038 0.105"/>
-        </geometry>
+          <mesh filename="package://${MESH_LINK_2}"
+              scale="1 1 1"/>
+        </geometry>
+        <material name="black"/>
+      </visual>
+      <collision>
+        <origin xyz="0 0 0" rpy="${M_PI/2} 0 0"/>
+        <geometry>
+          <mesh filename="package://${MESH_COLLISION_LINK_2}"
+              scale="1 1 1"/>
+        </geometry>
+        <material name="black"/>
       </collision>
       <inertial>
@@ -158,14 +176,16 @@
         <origin xyz="0 0 0" rpy="${M_PI/2} 0 0"/>
         <geometry>
-          <mesh filename="package://crane_plus_description/meshes/visual/RT-CRANE+_Link3.stl"
-              scale="1 1 1"/>
-        </geometry>
-        <material name="white"/>
-      </visual>
-      <collision>
-        <origin xyz="0 0 0.08" rpy="0 0 0"/>
-        <geometry>
-          <box size="0.032 0.035 0.050"/>
-        </geometry>
+          <mesh filename="package://${MESH_LINK_3}"
+              scale="1 1 1"/>
+        </geometry>
+        <material name="white"/>
+      </visual>
+      <collision>
+        <origin xyz="0 0 0" rpy="${M_PI/2} 0 0"/>
+        <geometry>
+          <mesh filename="package://${MESH_COLLISION_LINK_3}"
+              scale="1 1 1"/>
+        </geometry>
+        <material name="white"/>
       </collision>
       <inertial>
@@ -192,14 +212,16 @@
         <origin xyz="0 0 0" rpy="${M_PI/2} 0 0"/>
         <geometry>
-          <mesh filename="package://crane_plus_description/meshes/visual/RT-CRANE+_Link4.stl"
-              scale="1 1 1"/>
-        </geometry>
-        <material name="black"/>
-      </visual>
-      <collision>
-        <origin xyz="0 0.037 0.097" rpy="${M_PI/2} 0 0"/>
-        <geometry>
-          <box size="0.034 0.045 0.002"/>
-        </geometry>
+          <mesh filename="package://${MESH_LINK_4}"
+              scale="1 1 1"/>
+        </geometry>
+        <material name="black"/>
+      </visual>
+      <collision>
+        <origin xyz="0 0 0" rpy="${M_PI/2} 0 0"/>
+        <geometry>
+          <mesh filename="package://${MESH_COLLISION_LINK_4}"
+              scale="1 1 1"/>
+        </geometry>
+        <material name="black"/>
       </collision>
       <inertial>
@@ -226,14 +248,16 @@
         <origin xyz="0 0 0" rpy="0 -${M_PI/2} 0"/>
         <geometry>
-          <mesh filename="package://crane_plus_description/meshes/visual/RT-CRANE+_Hand.stl"
-              scale="1 1 1"/>
-        </geometry>
-        <material name="white"/>
-      </visual>
-      <collision>
-        <origin xyz="0 -0.018 0.075" rpy="${M_PI/3} 0 0"/>
-        <geometry>
-          <box size="0.034 0.045 0.002"/>
-        </geometry>
+          <mesh filename="package://${MESH_LINK_HAND}"
+              scale="1 1 1"/>
+        </geometry>
+        <material name="white"/>
+      </visual>
+      <collision>
+        <origin xyz="0 0 0" rpy="0 -${M_PI/2} 0"/>
+        <geometry>
+          <mesh filename="package://${MESH_COLLISION_LINK_HAND}"
+              scale="1 1 1"/>
+        </geometry>
+        <material name="white"/>
       </collision>
       <inertial>
