Commit message: Use new ros2 control interface (#27)
* Use new ros2_control API

* Delete unused files

* update comments

* Read joint speeds

* Change update _rate to 100Hz

* Disable read joint speeds to avoid a decrease of the communication rate.

* fix package.xml

* Refactoring crane_plus_driver

* Driver can read joint load, voltage and temperature

* Get dyanmixel id from joint's parameter

* Refactoring

* Fic container_ci.yml

* Update installation

* Use controller spawner to load controllers

* Add parameters to arm and gripper controller for trajectory control

* Add options for reading servo parameters

* Update crane_plus_control's README

* Change to print a communication timeout message once

* Reformat via ament-uncrustify

* Load ros2_control.xacro from crane_plus.xacro. This makes using gazebo_ros2_control easier.

* Use steady timer for timeout detection

* Pcrane_plus_drivers's functions use references instead of pointers

* Update crane_plus_control/README.md

* Update Installation

* Rename read_xbyte_list to read_xbyte_data_from_each_joints

* Refactor launch file

* Rename 1byte to byte, 2byte to word

* Refacotring to pass lint check

File: crane_plus_description/urdf/crane_plus.xacro (robot description, xacro)
@@ -21,16 +21,4 @@
   <xacro:property name="SCALE_MM" value="0.001"/>
   <xacro:property name="SCALE_CM" value="0.01"/>
-  <xacro:property name="NAME_JOINT_BASE" value="crane_plus_joint_base"/>
-  <xacro:property name="NAME_JOINT_1" value="crane_plus_joint1"/>
-  <xacro:property name="NAME_JOINT_2" value="crane_plus_joint2"/>
-  <xacro:property name="NAME_JOINT_3" value="crane_plus_joint3"/>
-  <xacro:property name="NAME_JOINT_4" value="crane_plus_joint4"/>
-  <xacro:property name="NAME_JOINT_HAND" value="crane_plus_joint_hand"/>
-  <xacro:property name="NAME_LINK_BASE" value="crane_plus_base"/>
-  <xacro:property name="NAME_LINK_1" value="crane_plus_link1"/>
-  <xacro:property name="NAME_LINK_2" value="crane_plus_link2"/>
-  <xacro:property name="NAME_LINK_3" value="crane_plus_link3"/>
-  <xacro:property name="NAME_LINK_4" value="crane_plus_link4"/>
-  <xacro:property name="NAME_LINK_HAND" value="crane_plus_link_hand"/>
   <xacro:property name="MESH_LINK_BASE" value="crane_plus_description/meshes/visual/body_20201013.stl"/>
   <xacro:property name="MESH_LINK_1" value="crane_plus_description/meshes/visual/Link1_20201013.stl"/>
@@ -47,22 +35,34 @@
   <xacro:macro name="crane_plus"
       params="parent
+              name_link_base
+              name_link_1
+              name_link_2
+              name_link_3
+              name_link_4
+              name_link_hand
+              name_joint_base
+              name_joint_1
+              name_joint_2
+              name_joint_3
+              name_joint_4
+              name_joint_hand
               joints_vlimit
-              joint1_lower_limit
-              joint1_upper_limit
-              joint2_lower_limit
-              joint2_upper_limit
-              joint3_lower_limit
-              joint3_upper_limit
-              joint4_lower_limit
-              joint4_upper_limit
+              joint_1_lower_limit
+              joint_1_upper_limit
+              joint_2_lower_limit
+              joint_2_upper_limit
+              joint_3_lower_limit
+              joint_3_upper_limit
+              joint_4_lower_limit
+              joint_4_upper_limit
               joint_hand_lower_limit
               joint_hand_upper_limit
               *origin">
-    <joint name="${NAME_JOINT_BASE}" type="fixed">
+    <joint name="${name_joint_base}" type="fixed">
       <xacro:insert_block name="origin"/>
       <parent link="${parent}"/>
-      <child link="${NAME_LINK_BASE}"/>
-    </joint>
-    <link name="${NAME_LINK_BASE}">
+      <child link="${name_link_base}"/>
+    </joint>
+    <link name="${name_link_base}">
       <visual>
         <origin xyz="0 0 0" rpy="0 0 0"/>
@@ -87,5 +87,5 @@
       </inertial>
     </link>
-    <joint name="${NAME_JOINT_1}" type="revolute">
+    <joint name="${name_joint_1}" type="revolute">
       <origin xyz="0 0 0.0454" rpy="0 0 0"/>
       <axis xyz="0 0 1"/>
@@ -93,12 +93,12 @@
         effort="10.0"
         velocity="${joints_vlimit}"
-        lower="${joint1_lower_limit}"
-        upper="${joint1_upper_limit}"
-        />
-      <parent link="${NAME_LINK_BASE}"/>
-      <child link="${NAME_LINK_1}"/>
-      <dynamics damping="1.0e-6" friction="2.0e-1"/>
-    </joint>
-    <link name="${NAME_LINK_1}">
+        lower="${joint_1_lower_limit}"
+        upper="${joint_1_upper_limit}"
+        />
+      <parent link="${name_link_base}"/>
+      <child link="${name_link_1}"/>
+      <dynamics damping="1.0e-6" friction="2.0e-1"/>
+    </joint>
+    <link name="${name_link_1}">
       <visual>
         <origin xyz="0 0 0" rpy="0 0 ${M_PI}"/>
@@ -123,5 +123,5 @@
       </inertial>
     </link>
-    <joint name="${NAME_JOINT_2}" type="revolute">
+    <joint name="${name_joint_2}" type="revolute">
       <origin xyz="0 0 0.026" rpy="0 0 0"/>
       <axis xyz="0 1 0"/>
@@ -129,12 +129,12 @@
         effort="10.0"
         velocity="${joints_vlimit}"
-        lower="${joint2_lower_limit}"
-        upper="${joint2_upper_limit}"
-        />
-      <parent link="${NAME_LINK_1}"/>
-      <child link="${NAME_LINK_2}"/>
-      <dynamics damping="1.0e-6" friction="2.0e-1"/>
-    </joint>
-    <link name="${NAME_LINK_2}">
+        lower="${joint_2_lower_limit}"
+        upper="${joint_2_upper_limit}"
+        />
+      <parent link="${name_link_1}"/>
+      <child link="${name_link_2}"/>
+      <dynamics damping="1.0e-6" friction="2.0e-1"/>
+    </joint>
+    <link name="${name_link_2}">
       <visual>
         <origin xyz="0 0 0" rpy="${M_PI/2} 0 0"/>
@@ -159,5 +159,5 @@
       </inertial>
     </link>
-    <joint name="${NAME_JOINT_3}" type="revolute">
+    <joint name="${name_joint_3}" type="revolute">
       <origin xyz="0 0 0.083" rpy="0 0 0"/>
       <axis xyz="0 -1 0"/>
@@ -165,12 +165,12 @@
         effort="10.0"
         velocity="${joints_vlimit}"
-        lower="${joint3_lower_limit}"
-        upper="${joint3_upper_limit}"
-        />
-      <parent link="${NAME_LINK_2}"/>
-      <child link="${NAME_LINK_3}"/>
-      <dynamics damping="1.0e-6" friction="2.0e-1"/>
-    </joint>
-    <link name="${NAME_LINK_3}">
+        lower="${joint_3_lower_limit}"
+        upper="${joint_3_upper_limit}"
+        />
+      <parent link="${name_link_2}"/>
+      <child link="${name_link_3}"/>
+      <dynamics damping="1.0e-6" friction="2.0e-1"/>
+    </joint>
+    <link name="${name_link_3}">
       <visual>
         <origin xyz="0 0 0" rpy="${M_PI/2} 0 0"/>
@@ -195,5 +195,5 @@
       </inertial>
     </link>
-    <joint name="${NAME_JOINT_4}" type="revolute">
+    <joint name="${name_joint_4}" type="revolute">
       <origin xyz="0 0 0.0935" rpy="0 0 0"/>
       <axis xyz="0 -1 0"/>
@@ -201,12 +201,12 @@
         effort="10.0"
         velocity="${joints_vlimit}"
-        lower="${joint4_lower_limit}"
-        upper="${joint4_upper_limit}"
-        />
-      <parent link="${NAME_LINK_3}"/>
-      <child link="${NAME_LINK_4}"/>
-      <dynamics damping="1.0e-6" friction="2.0e-1"/>
-    </joint>
-    <link name="${NAME_LINK_4}">
+        lower="${joint_4_lower_limit}"
+        upper="${joint_4_upper_limit}"
+        />
+      <parent link="${name_link_3}"/>
+      <child link="${name_link_4}"/>
+      <dynamics damping="1.0e-6" friction="2.0e-1"/>
+    </joint>
+    <link name="${name_link_4}">
       <visual>
         <origin xyz="0 0 0" rpy="${M_PI/2} 0 0"/>
@@ -231,5 +231,5 @@
       </inertial>
     </link>
-    <joint name="${NAME_JOINT_HAND}" type="revolute">
+    <joint name="${name_joint_hand}" type="revolute">
       <origin xyz="0 -0.0145 0.045" rpy="0 0 0"/>
       <axis xyz="-1 0 0"/>
@@ -240,9 +240,9 @@
         upper="${joint_hand_upper_limit}"
         />
-      <parent link="${NAME_LINK_4}"/>
-      <child link="${NAME_LINK_HAND}"/>
-      <dynamics damping="1.0e-6" friction="2.0e-1"/>
-    </joint>
-    <link name="${NAME_LINK_HAND}">
+      <parent link="${name_link_4}"/>
+      <child link="${name_link_hand}"/>
+      <dynamics damping="1.0e-6" friction="2.0e-1"/>
+    </joint>
+    <link name="${name_link_hand}">
       <visual>
         <origin xyz="0 0 0" rpy="0 -${M_PI/2} 0"/>

Commit message: 不要なマテリアルを削除

File: crane_plus_description/urdf/crane_plus.xacro (robot description, xacro)
@@ -6,16 +6,4 @@
   <material name="white">
     <color rgba="0.95 0.95 0.95 1.0"/>
-  </material>
-  <material name="silver">
-    <color rgba="0.75 0.75 0.75 1.0"/>
-  </material>
-  <material name="red">
-    <color rgba="1.0 0.3 0.3 1.0"/>
-  </material>
-  <material name="green">
-    <color rgba="0.3 1.0 0.3 1.0"/>
-  </material>
-  <material name="blue">
-    <color rgba="0.3 0.3 1.0 1.0"/>
   </material>
   <xacro:property name="SCALE_MM" value="0.001"/>

Commit message: 使用していないSCALEの変数を削除

File: crane_plus_description/urdf/crane_plus.xacro (robot description, xacro)
@@ -7,6 +7,4 @@
     <color rgba="0.95 0.95 0.95 1.0"/>
   </material>
-  <xacro:property name="SCALE_MM" value="0.001"/>
-  <xacro:property name="SCALE_CM" value="0.01"/>
   <xacro:property name="MESH_LINK_BASE" value="crane_plus_description/meshes/visual/body_20201013.stl"/>
   <xacro:property name="MESH_LINK_1" value="crane_plus_description/meshes/visual/Link1_20201013.stl"/>

Commit message: STLファイルのパスを直書きに修正

File: crane_plus_description/urdf/crane_plus.xacro (robot description, xacro)
@@ -55,6 +55,5 @@
         <origin xyz="0 0 0" rpy="0 0 0"/>
         <geometry>
-          <mesh filename="package://${MESH_LINK_BASE}"
-              scale="1 1 1"/>
+          <mesh filename="package://crane_plus_description/meshes/visual/body_20201013.stl" scale="1 1 1"/>
         </geometry>
         <material name="black"/>
@@ -63,6 +62,5 @@
         <origin xyz="0 0 0" rpy="0 0 0"/>
         <geometry>
-          <mesh filename="package://${MESH_COLLISION_LINK_BASE}"
-              scale="1 1 1"/>
+          <mesh filename="package://crane_plus_description/meshes/collision/body_collision_20201013.stl" scale="1 1 1"/>
         </geometry>
         <material name="black"/>
@@ -91,6 +89,5 @@
         <origin xyz="0 0 0" rpy="0 0 ${M_PI}"/>
         <geometry>
-          <mesh filename="package://${MESH_LINK_1}"
-              scale="1 1 1"/>
+          <mesh filename="package://crane_plus_description/meshes/visual/Link1_20201013.stl" scale="1 1 1"/>
         </geometry>
         <material name="white"/>
@@ -99,6 +96,5 @@
         <origin xyz="0 0 0" rpy="0 0 ${M_PI}"/>
         <geometry>
-          <mesh filename="package://${MESH_COLLISION_LINK_1}"
-              scale="1 1 1"/>
+          <mesh filename="package://crane_plus_description/meshes/collision/Link1_collision_20201013.stl" scale="1 1 1"/>
         </geometry>
         <material name="white"/>
@@ -127,14 +123,12 @@
         <origin xyz="0 0 0" rpy="${M_PI/2} 0 0"/>
         <geometry>
-          <mesh filename="package://${MESH_LINK_2}"
-              scale="1 1 1"/>
-        </geometry>
-        <material name="black"/>
-      </visual>
-      <collision>
-        <origin xyz="0 0 0" rpy="${M_PI/2} 0 0"/>
-        <geometry>
-          <mesh filename="package://${MESH_COLLISION_LINK_2}"
-              scale="1 1 1"/>
+          <mesh filename="package://crane_plus_description/meshes/visual/Link2_20201013.stl" scale="1 1 1"/>
+        </geometry>
+        <material name="black"/>
+      </visual>
+      <collision>
+        <origin xyz="0 0 0" rpy="${M_PI/2} 0 0"/>
+        <geometry>
+          <mesh filename="package://crane_plus_description/meshes/collision/Link2_collision_20201013.stl" scale="1 1 1"/>
         </geometry>
         <material name="black"/>
@@ -163,14 +157,12 @@
         <origin xyz="0 0 0" rpy="${M_PI/2} 0 0"/>
         <geometry>
-          <mesh filename="package://${MESH_LINK_3}"
-              scale="1 1 1"/>
-        </geometry>
-        <material name="white"/>
-      </visual>
-      <collision>
-        <origin xyz="0 0 0" rpy="${M_PI/2} 0 0"/>
-        <geometry>
-          <mesh filename="package://${MESH_COLLISION_LINK_3}"
-              scale="1 1 1"/>
+          <mesh filename="package://crane_plus_description/meshes/visual/Link3_20201013.stl" scale="1 1 1"/>
+        </geometry>
+        <material name="white"/>
+      </visual>
+      <collision>
+        <origin xyz="0 0 0" rpy="${M_PI/2} 0 0"/>
+        <geometry>
+          <mesh filename="package://crane_plus_description/meshes/collision/Link3_collision_20201013.stl" scale="1 1 1"/>
         </geometry>
         <material name="white"/>
@@ -199,14 +191,12 @@
         <origin xyz="0 0 0" rpy="${M_PI/2} 0 0"/>
         <geometry>
-          <mesh filename="package://${MESH_LINK_4}"
-              scale="1 1 1"/>
-        </geometry>
-        <material name="black"/>
-      </visual>
-      <collision>
-        <origin xyz="0 0 0" rpy="${M_PI/2} 0 0"/>
-        <geometry>
-          <mesh filename="package://${MESH_COLLISION_LINK_4}"
-              scale="1 1 1"/>
+          <mesh filename="package://crane_plus_description/meshes/visual/Link4_20201013.stl" scale="1 1 1"/>
+        </geometry>
+        <material name="black"/>
+      </visual>
+      <collision>
+        <origin xyz="0 0 0" rpy="${M_PI/2} 0 0"/>
+        <geometry>
+          <mesh filename="package://crane_plus_description/meshes/collision/Link4_collision_20201013.stl" scale="1 1 1"/>
         </geometry>
         <material name="black"/>
@@ -235,6 +225,5 @@
         <origin xyz="0 0 0" rpy="0 -${M_PI/2} 0"/>
         <geometry>
-          <mesh filename="package://${MESH_LINK_HAND}"
-              scale="1 1 1"/>
+          <mesh filename="package://crane_plus_description/meshes/visual/Hand_20201013.stl" scale="1 1 1"/>
         </geometry>
         <material name="white"/>
@@ -243,6 +232,5 @@
         <origin xyz="0 0 0" rpy="0 -${M_PI/2} 0"/>
         <geometry>
-          <mesh filename="package://${MESH_COLLISION_LINK_HAND}"
-              scale="1 1 1"/>
+          <mesh filename="package://crane_plus_description/meshes/collision/Hand_collision_20201013.stl" scale="1 1 1"/>
         </geometry>
         <material name="white"/>

Commit message: STLファイルのパスの変数を削除

File: crane_plus_description/urdf/crane_plus.xacro (robot description, xacro)
@@ -7,16 +7,4 @@
     <color rgba="0.95 0.95 0.95 1.0"/>
   </material>
-  <xacro:property name="MESH_LINK_BASE" value="crane_plus_description/meshes/visual/body_20201013.stl"/>
-  <xacro:property name="MESH_LINK_1" value="crane_plus_description/meshes/visual/Link1_20201013.stl"/>
-  <xacro:property name="MESH_LINK_2" value="crane_plus_description/meshes/visual/Link2_20201013.stl"/>
-  <xacro:property name="MESH_LINK_3" value="crane_plus_description/meshes/visual/Link3_20201013.stl"/>
-  <xacro:property name="MESH_LINK_4" value="crane_plus_description/meshes/visual/Link4_20201013.stl"/>
-  <xacro:property name="MESH_LINK_HAND" value="crane_plus_description/meshes/visual/Hand_20201013.stl"/>
-  <xacro:property name="MESH_COLLISION_LINK_BASE" value="crane_plus_description/meshes/collision/body_collision_20201013.stl"/>
-  <xacro:property name="MESH_COLLISION_LINK_1" value="crane_plus_description/meshes/collision/Link1_collision_20201013.stl"/>
-  <xacro:property name="MESH_COLLISION_LINK_2" value="crane_plus_description/meshes/collision/Link2_collision_20201013.stl"/>
-  <xacro:property name="MESH_COLLISION_LINK_3" value="crane_plus_description/meshes/collision/Link3_collision_20201013.stl"/>
-  <xacro:property name="MESH_COLLISION_LINK_4" value="crane_plus_description/meshes/collision/Link4_collision_20201013.stl"/>
-  <xacro:property name="MESH_COLLISION_LINK_HAND" value="crane_plus_description/meshes/collision/Hand_collision_20201013.stl"/>
   <xacro:macro name="crane_plus"
       params="parent

Commit message: 各リンクのinertialを修正

File: crane_plus_description/urdf/crane_plus.xacro (robot description, xacro)
@@ -55,6 +55,6 @@
       </collision>
       <inertial>
-        <mass value="0.06645"/>
-        <origin xyz="-1.31E-02 7.00E-06 2.12E-02" rpy="0 ${M_PI/8} 0"/>
+        <mass value="6.65E-02"/>
+        <origin xyz="-1.31E-02 7.00E-06 2.12E-02" rpy="0 0 0"/>
         <inertia ixx="1.66E-05" ixy="1.80E-09" ixz="-5.75E-07" iyy="2.36E-05" iyz="-3.23E-08" izz="1.77E-05"/>
       </inertial>
@@ -89,5 +89,5 @@
       </collision>
       <inertial>
-        <mass value="0.007729"/>
+        <mass value="7.73E-03"/>
         <origin xyz="2.00E-06 0.0 1.09E-02" rpy="0 0 0"/>
         <inertia ixx="3.43E-06" ixy="0.0" ixz="1.66E-10" iyy="1.30E-06" iyz="0.0" izz="3.05E-06"/>
@@ -123,5 +123,5 @@
       </collision>
       <inertial>
-        <mass value="0.116745"/>
+        <mass value="1.17E-01"/>
         <origin xyz="7.99E-04 1.00E-06 4.15E-02" rpy="${M_PI/2} 0 0"/>
         <inertia ixx="1.25E-04" ixy="6.83E-08" ixz="9.50E-11" iyy="1.92E-05" iyz="0.0" izz="1.19E-04"/>
@@ -157,5 +157,5 @@
       </collision>
       <inertial>
-        <mass value="0.072317"/>
+        <mass value="7.23E-02"/>
         <origin xyz="6.45E-04 -1.38E-04 7.01E-02" rpy="${M_PI/2} 0 0"/>
         <inertia ixx="5.41E-05" ixy="-2.28E-07" ixz="-2.67E-09" iyy="1.60E-05" iyz="-5.35E-07" izz="4.69E-05"/>
@@ -191,5 +191,5 @@
       </collision>
       <inertial>
-        <mass value="0.08185"/>
+        <mass value="8.19E-02"/>
         <origin xyz="6.45E-04 -5.70E-04 4.62E-02" rpy="${M_PI/2} 0 0"/>
         <inertia ixx="5.91E-05" ixy="-5.11E-08" ixz="3.49E-07" iyy="3.62E-05" iyz="1.37E-05" izz="3.98E-05"/>
@@ -225,6 +225,6 @@
       </collision>
       <inertial>
-        <mass value="0.022901"/>
-        <origin xyz="0.0 -2.04E-02 2.77E-02" rpy="0 ${M_PI/2} 0"/>
+        <mass value="2.29E-02"/>
+        <origin xyz="0.0 -2.04E-02 2.77E-02" rpy="0 -${M_PI/2} 0"/>
         <inertia ixx="5.76E-06" ixy="-4.66E-07" ixz="0.0" iyy="2.76E-05" iyz="0.0" izz="2.52E-05"/>
       </inertial>
