Commit message: stlファイルの名前をシンプルに修正

File: crane_plus_description/urdf/crane_plus.xacro (robot description, xacro)
@@ -11,12 +11,12 @@
         <origin xyz="0 0 0" rpy="0 0 0"/>
         <geometry>
-          <mesh filename="package://crane_plus_description/meshes/visual/body_20201013.stl" scale="1 1 1"/>
-        </geometry>
-        <material name="black"/>
-      </visual>
-      <collision>
-        <origin xyz="0 0 0" rpy="0 0 0"/>
-        <geometry>
-          <mesh filename="package://crane_plus_description/meshes/collision/body_collision_20201013.stl" scale="1 1 1"/>
+          <mesh filename="package://crane_plus_description/meshes/visual/body.stl" scale="1 1 1"/>
+        </geometry>
+        <material name="black"/>
+      </visual>
+      <collision>
+        <origin xyz="0 0 0" rpy="0 0 0"/>
+        <geometry>
+          <mesh filename="package://crane_plus_description/meshes/collision/body.stl" scale="1 1 1"/>
         </geometry>
         <material name="black"/>
@@ -45,12 +45,12 @@
         <origin xyz="0 0 0" rpy="0 0 0"/>
         <geometry>
-          <mesh filename="package://crane_plus_description/meshes/visual/Link1_20201013.stl" scale="1 1 1"/>
-        </geometry>
-        <material name="white"/>
-      </visual>
-      <collision>
-        <origin xyz="0 0 0" rpy="0 0 0"/>
-        <geometry>
-          <mesh filename="package://crane_plus_description/meshes/collision/Link1_collision_20201013.stl" scale="1 1 1"/>
+          <mesh filename="package://crane_plus_description/meshes/visual/link1.stl" scale="1 1 1"/>
+        </geometry>
+        <material name="white"/>
+      </visual>
+      <collision>
+        <origin xyz="0 0 0" rpy="0 0 0"/>
+        <geometry>
+          <mesh filename="package://crane_plus_description/meshes/collision/link1.stl" scale="1 1 1"/>
         </geometry>
         <material name="white"/>
@@ -79,12 +79,12 @@
         <origin xyz="0 0 0" rpy="${radians(90)} 0 0"/>
         <geometry>
-          <mesh filename="package://crane_plus_description/meshes/visual/Link2_20201013.stl" scale="1 1 1"/>
-        </geometry>
-        <material name="black"/>
-      </visual>
-      <collision>
-        <origin xyz="0 0 0" rpy="${radians(90)} 0 0"/>
-        <geometry>
-          <mesh filename="package://crane_plus_description/meshes/collision/Link2_collision_20201013.stl" scale="1 1 1"/>
+          <mesh filename="package://crane_plus_description/meshes/visual/link2.stl" scale="1 1 1"/>
+        </geometry>
+        <material name="black"/>
+      </visual>
+      <collision>
+        <origin xyz="0 0 0" rpy="${radians(90)} 0 0"/>
+        <geometry>
+          <mesh filename="package://crane_plus_description/meshes/collision/link2.stl" scale="1 1 1"/>
         </geometry>
         <material name="black"/>
@@ -113,12 +113,12 @@
         <origin xyz="0 0 0" rpy="${radians(90)} 0 0"/>
         <geometry>
-          <mesh filename="package://crane_plus_description/meshes/visual/Link3_20201013.stl" scale="1 1 1"/>
-        </geometry>
-        <material name="white"/>
-      </visual>
-      <collision>
-        <origin xyz="0 0 0" rpy="${radians(90)} 0 0"/>
-        <geometry>
-          <mesh filename="package://crane_plus_description/meshes/collision/Link3_collision_20201013.stl" scale="1 1 1"/>
+          <mesh filename="package://crane_plus_description/meshes/visual/link3.stl" scale="1 1 1"/>
+        </geometry>
+        <material name="white"/>
+      </visual>
+      <collision>
+        <origin xyz="0 0 0" rpy="${radians(90)} 0 0"/>
+        <geometry>
+          <mesh filename="package://crane_plus_description/meshes/collision/link3.stl" scale="1 1 1"/>
         </geometry>
         <material name="white"/>
@@ -147,12 +147,12 @@
         <origin xyz="0 0 0" rpy="${radians(90)} 0 0"/>
         <geometry>
-          <mesh filename="package://crane_plus_description/meshes/visual/Link4_20201013.stl" scale="1 1 1"/>
-        </geometry>
-        <material name="black"/>
-      </visual>
-      <collision>
-        <origin xyz="0 0 0" rpy="${radians(90)} 0 0"/>
-        <geometry>
-          <mesh filename="package://crane_plus_description/meshes/collision/Link4_collision_20201013.stl" scale="1 1 1"/>
+          <mesh filename="package://crane_plus_description/meshes/visual/link4.stl" scale="1 1 1"/>
+        </geometry>
+        <material name="black"/>
+      </visual>
+      <collision>
+        <origin xyz="0 0 0" rpy="${radians(90)} 0 0"/>
+        <geometry>
+          <mesh filename="package://crane_plus_description/meshes/collision/link4.stl" scale="1 1 1"/>
         </geometry>
         <material name="black"/>
@@ -181,5 +181,5 @@
         <origin xyz="0 0 0" rpy="0 ${radians(-90)} 0"/>
         <geometry>
-          <mesh filename="package://crane_plus_description/meshes/visual/Hand_20201013.stl" scale="1 1 1"/>
+          <mesh filename="package://crane_plus_description/meshes/visual/hand.stl" scale="1 1 1"/>
         </geometry>
         <material name="white"/>
@@ -188,5 +188,5 @@
         <origin xyz="0 0 0" rpy="0 ${radians(-90)} 0"/>
         <geometry>
-          <mesh filename="package://crane_plus_description/meshes/collision/Hand_collision_20201013.stl" scale="1 1 1"/>
+          <mesh filename="package://crane_plus_description/meshes/collision/hand.stl" scale="1 1 1"/>
         </geometry>
         <material name="white"/>

Commit message: TCPリンクの位置を0.121mに変更

File: crane_plus_description/urdf/crane_plus.xacro (robot description, xacro)
@@ -199,5 +199,5 @@
     </link>
     <joint name="${NAME_JOINT_TCP}" type="fixed">
-      <origin xyz="0 0 0.09" rpy="0 0 0"/>
+      <origin xyz="0 0 0.121" rpy="0 0 0"/>
       <parent link="${NAME_LINK_4}"/>
       <child link="${NAME_LINK_TCP}"/>
